Commit message: Added grips_manipulation package to support collision free motion

File: grips_description/robots/grips.xacro (robot description, xacro)
@@ -1,4 +1,4 @@
 <?xml version="1.0"?>
-<robot name="grips" xmlns:xacro="http://www.ros.org/wiki/xacro">
+<robot name="grips_simple_gripper" xmlns:xacro="http://www.ros.org/wiki/xacro">
 	<!-- Import common macros-->
 	<xacro:include filename="$(find grips_description)/urdf/common.xacro" />
@@ -7,4 +7,6 @@
 	<!-- Import robot without gripper -->
 	<xacro:include filename="$(find grips_description)/urdf/grips.xacro" />
+	<!-- Import simple gripper -->
+	<xacro:include filename="$(find grips_description)/urdf/simple_gripper.xacro" />
 	<!-- Used for fixing robot to Gazebo 'base_link' -->
 	<link name="world" />
@@ -14,3 +16,18 @@
 		<child link="base_link" />
 	</joint>
+	<!-- Used for fixing the gripper to the robot -->
+	<joint name="gripper_anchor" type="fixed">
+		<origin xyz="0 0 0" rpy="0 0 0" />
+		<parent link="end_effector" />
+		<child link="gripper_base" />
+	</joint>
+	<!-- ros_control plugin -->
+	<gazebo>
+		<plugin name="ros_control" filename="libgazebo_ros_control.so">
+<!--
+			<robotNamespace>/grips_simple_gripper</robotNamespace>
+      <robotParam>/grips_simple_gripper/robot_description</robotParam>
+-->
+		</plugin>
+	</gazebo>
 </robot>
