Commit message: Multi-robots configurations supported. Requieres this two pull requests: - https://github.com/ros-controls/ros_controllers/pull/57 - https://github.com/piyushk/robot_state_publisher/pull/1

File: grips_description/robots/grips.urdf (robot description, URDF)
Before this commit: robot grips, 11 links, 10 joints
Links:
- link base_link: geometry collision mesh filename=package://grips_description/meshes/base/base_collision.dae; visual mesh filename=package://grips_description/meshes/base/base.dae
- link camera_link: geometry collision mesh filename=package://grips_description/meshes/camera/camera_collision.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; visual mesh filename=package://grips_description/meshes/camera/camera.dae
- link coupling_link: geometry collision mesh filename=package://grips_description/meshes/linkage/coupling.dae; visual mesh filename=package://grips_description/meshes/linkage/coupling.dae
- link elbow_pivot_link: geometry collision mesh filename=package://grips_description/meshes/linkage/elbow_pivot.dae; visual mesh filename=package://grips_description/meshes/linkage/elbow_pivot.dae
- link forearm_link: geometry collision mesh filename=package://grips_description/meshes/forearm/forearm_collisio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; visual mesh filename=package://grips_description/meshes/forearm/forearm.dae
- link manifold_link: geometry collision mesh filename=package://grips_description/meshes/manifold/manifold_collis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; visual mesh filename=package://grips_description/meshes/manifold/manifold.dae
- link pitch_link: geometry collision mesh filename=package://grips_description/meshes/pitch/pitch_collision.dae; visual mesh filename=package://grips_description/meshes/pitch/pitch.dae
- link upper_arm_link: geometry collision mesh filename=package://grips_description/meshes/upper_arm/upper_arm_coll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; visual mesh filename=package://grips_description/meshes/upper_arm/upper_arm.dae
- link yaw_link: geometry collision mesh filename=package://grips_description/meshes/yaw/yaw_collision.dae; visual mesh filename=package://grips_description/meshes/yaw/yaw.dae

File: grips_description/robots/grips_simple_gripper.urdf (robot description, URDF)
Before this commit: robot grips_simple_gripper, 18 links, 17 joints
Links:
- link base_link: geometry collision mesh filename=package://grips_description/meshes/base/base_collision.dae; visual mesh filename=package://grips_description/meshes/base/base.dae
- link camera_link: geometry collision mesh filename=package://grips_description/meshes/camera/camera_collision.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; visual mesh filename=package://grips_description/meshes/camera/camera.dae
- link coupling_link: geometry collision mesh filename=package://grips_description/meshes/linkage/coupling.dae; visual mesh filename=package://grips_description/meshes/linkage/coupling.dae
- link elbow_pivot_link: geometry collision mesh filename=package://grips_description/meshes/linkage/elbow_pivot.dae; visual mesh filename=package://grips_description/meshes/linkage/elbow_pivot.dae
- link forearm_link: geometry collision mesh filename=package://grips_description/meshes/forearm/forearm_collisio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; visual mesh filename=package://grips_description/meshes/forearm/forearm.dae
- link gripper_base: geometry collision mesh filename=package://grips_description/meshes/gripper/gripper_base.dae; visual mesh filename=package://grips_description/meshes/gripper/gripper_base.dae
- link l_finger_link: geometry collision mesh filename=package://grips_description/meshes/gripper/l_finger.dae; visual mesh filename=package://grips_description/meshes/gripper/l_finger.dae
- link l_inner_link: geometry collision mesh filename=package://grips_description/meshes/gripper/l_inner_pivot.dae; visual mesh filename=package://grips_description/meshes/gripper/l_inner_pivot.dae
- link l_outer_link: geometry collision mesh filename=package://grips_description/meshes/gripper/outer_pivot.dae; visual mesh filename=package://grips_description/meshes/gripper/outer_pivot.dae
- link manifold_link: geometry collision mesh filename=package://grips_description/meshes/manifold/manifold_collis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; visual mesh filename=package://grips_description/meshes/manifold/manifold.dae
- link pitch_link: geometry collision mesh filename=package://grips_description/meshes/pitch/pitch_collision.dae; visual mesh filename=package://grips_description/meshes/pitch/pitch.dae
- link r_finger_link: geometry collision mesh filename=package://grips_description/meshes/gripper/r_finger.dae; visual mesh filename=package://grips_description/meshes/gripper/r_finger.dae
- link r_inner_link: geometry collision mesh filename=package://grips_description/meshes/gripper/r_inner_pivot.dae; visual mesh filename=package://grips_description/meshes/gripper/r_inner_pivot.dae
- link r_outer_link: geometry collision mesh filename=package://grips_description/meshes/gripper/outer_pivot.dae; visual mesh filename=package://grips_description/meshes/gripper/outer_pivot.dae
- link upper_arm_link: geometry collision mesh filename=package://grips_description/meshes/upper_arm/upper_arm_coll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; visual mesh filename=package://grips_description/meshes/upper_arm/upper_arm.dae
- link yaw_link: geometry collision mesh filename=package://grips_description/meshes/yaw/yaw_collision.dae; visual mesh filename=package://grips_description/meshes/yaw/yaw.dae

File: grips_description/robots/left_arm.xacro (robot description, xacro)
@@ -1,4 +1,4 @@
 <?xml version="1.0"?>
-<robot name="grips_simple_gripper" xmlns:xacro="http://www.ros.org/wiki/xacro">
+<robot name="left_arm" xmlns:xacro="http://www.ros.org/wiki/xacro">
 	<!-- Import common macros-->
 	<xacro:include filename="$(find grips_description)/urdf/common.xacro" />
@@ -12,5 +12,5 @@
 	<link name="world" />
 	<joint name="anchor" type="fixed">
-		<origin xyz="0 0 0.001" rpy="0 0 0" />
+		<origin xyz="0 0 0.801" rpy="0 0 0" />
 		<parent link="world" />
 		<child link="base_link" />
@@ -25,6 +25,6 @@
 	<gazebo>
 		<plugin name="ros_control" filename="libgazebo_ros_control.so">
-			<robotNamespace>/grips_simple_gripper</robotNamespace>
-      <robotParam>/grips_simple_gripper/robot_description</robotParam>
+			<robotNamespace>/left_arm</robotNamespace>
+      <robotParam>/left_arm/robot_description</robotParam>
 		</plugin>
 	</gazebo>

File: grips_description/robots/right_arm.xacro (robot description, xacro)
@@ -1,4 +1,4 @@
 <?xml version="1.0"?>
-<robot name="grips_simple_gripper" xmlns:xacro="http://www.ros.org/wiki/xacro">
+<robot name="right_arm" xmlns:xacro="http://www.ros.org/wiki/xacro">
 	<!-- Import common macros-->
 	<xacro:include filename="$(find grips_description)/urdf/common.xacro" />
@@ -12,5 +12,5 @@
 	<link name="world" />
 	<joint name="anchor" type="fixed">
-		<origin xyz="0 0 0.001" rpy="0 0 0" />
+		<origin xyz="1 0 0.801" rpy="0 0 0" />
 		<parent link="world" />
 		<child link="base_link" />
@@ -25,6 +25,6 @@
 	<gazebo>
 		<plugin name="ros_control" filename="libgazebo_ros_control.so">
-			<robotNamespace>/grips_simple_gripper</robotNamespace>
-      <robotParam>/grips_simple_gripper/robot_description</robotParam>
+			<robotNamespace>/right_arm</robotNamespace>
+      <robotParam>/right_arm/robot_description</robotParam>
 		</plugin>
 	</gazebo>

File: grips_description/urdf/common.xacro (robot description, xacro)
@@ -22,4 +22,24 @@
 		</link>
 	</macro>
+  <macro name="link_collision" params="name color mesh mass cog *collision *inertia">
+		<link name="${name}">
+			<visual>
+				<geometry>
+					<mesh filename="${mesh}" />
+				</geometry>
+				<material name="${color}" />
+			</visual>
+			<collision>
+				<geometry>
+					<xacro:insert_block name="collision" />
+				</geometry>
+			</collision>
+			<inertial>
+				<origin xyz="${cog}" rpy="0 0 0" />
+				<mass value="${mass}" />
+				<xacro:insert_block name="inertia" />
+			</inertial>
+		</link>
+	</macro>
 	<!-- Transmission's Macro -->
 	<macro name="simple_transmission" params="joint">

File: grips_description/urdf/grips.xacro (robot description, xacro)
@@ -73,13 +73,13 @@
 	</macro>
 	<!-- Meshes -->
-	<property name="base_mesh" value="package://grips_description/meshes/base.dae" />
-	<property name="manifold_mesh" value="package://grips_description/meshes/manifold.dae" />
-	<property name="upper_arm_mesh" value="package://grips_description/meshes/upper_arm.dae" />
-	<property name="elbow_pivot_mesh" value="package://grips_description/meshes/elbow_pivot.dae" />
-	<property name="coupling_mesh" value="package://grips_description/meshes/coupling.dae" />
-	<property name="forearm_mesh" value="package://grips_description/meshes/forearm.dae" />
-	<property name="pitch_mesh" value="package://grips_description/meshes/pitch.dae" />
-	<property name="yaw_mesh" value="package://grips_description/meshes/yaw.dae" />
-	<property name="camera_mesh" value="package://grips_description/meshes/camera.dae" />
+	<property name="base_mesh" value="package://grips_description/meshes/base/base.dae" />
+	<property name="manifold_mesh" value="package://grips_description/meshes/manifold/manifold.dae" />
+	<property name="upper_arm_mesh" value="package://grips_description/meshes/upper_arm/upper_arm.dae" />
+	<property name="elbow_pivot_mesh" value="package://grips_description/meshes/linkage/elbow_pivot.dae" />
+	<property name="coupling_mesh" value="package://grips_description/meshes/linkage/coupling.dae" />
+	<property name="forearm_mesh" value="package://grips_description/meshes/forearm/forearm.dae" />
+	<property name="pitch_mesh" value="package://grips_description/meshes/pitch/pitch.dae" />
+	<property name="yaw_mesh" value="package://grips_description/meshes/yaw/yaw.dae" />
+	<property name="camera_mesh" value="package://grips_description/meshes/camera/camera.dae" />
 	<!-- Joints Dynamics -->
 	<property name="SA_damping" value="5" />
@@ -91,15 +91,18 @@
 	<property name="WR_damping" value="0.5" />
 	<!-- base link -->
-	<create_link name="base_link" color="black" mesh="${base_mesh}" cog="${base_cog}" mass="${base_mass}" >
+	<link_collision name="base_link" color="black" mesh="${base_mesh}" cog="${base_cog}" mass="${base_mass}" >
+    <mesh filename="package://grips_description/meshes/base/base_collision.dae" />
 		<base_inertia />
-	</create_link>
+	</link_collision>
 	<!-- manifold link -->
-	<create_link name="manifold_link" color="blue" mesh="${manifold_mesh}" cog="${manifold_cog}" mass="${manifold_mass}" >
+	<link_collision name="manifold_link" color="blue" mesh="${manifold_mesh}" cog="${manifold_cog}" mass="${manifold_mass}" >
+    <mesh filename="package://grips_description/meshes/manifold/manifold_collision.dae" />
 		<manifold_inertia />
-	</create_link>
+	</link_collision>
 	<!-- upper arm link -->
-	<create_link name="upper_arm_link" color="black" mesh="${upper_arm_mesh}" cog="${upper_arm_cog}" mass="${upper_arm_mass}" >
+	<link_collision name="upper_arm_link" color="black" mesh="${upper_arm_mesh}" cog="${upper_arm_cog}" mass="${upper_arm_mass}" >
+    <mesh filename="package://grips_description/meshes/upper_arm/upper_arm_collision.dae" />
 		<upper_arm_inertia />
-	</create_link>
+	</link_collision>
 	<!-- elbow pivot link -->
 	<create_link name="elbow_pivot_link" color="black" mesh="${elbow_pivot_mesh}" cog="${elbow_pivot_cog}" mass="${elbow_pivot_mass}" >
@@ -111,21 +114,25 @@
 	</create_link>
 	<!-- forearm link -->
-	<create_link name="forearm_link" color="black" mesh="${forearm_mesh}" cog="${forearm_cog}" mass="${forearm_mass}" >
+	<link_collision name="forearm_link" color="black" mesh="${forearm_mesh}" cog="${forearm_cog}" mass="${forearm_mass}" >
+    <mesh filename="package://grips_description/meshes/forearm/forearm_collision.dae" />
 		<forearm_inertia />
-	</create_link>
+	</link_collision>
 	<!-- pitch link -->
-	<create_link name="pitch_link" color="black" mesh="${pitch_mesh}" cog="${pitch_cog}" mass="${pitch_mass}" >
+	<link_collision name="pitch_link" color="black" mesh="${pitch_mesh}" cog="${pitch_cog}" mass="${pitch_mass}" >
+    <mesh filename="package://grips_description/meshes/pitch/pitch_collision.dae" />
 		<pitch_inertia />
-	</create_link>
+	</link_collision>
 	<!-- yaw link -->
-	<create_link name="yaw_link" color="black" mesh="${yaw_mesh}" cog="${yaw_cog}" mass="${yaw_mass}" >
+	<link_collision name="yaw_link" color="black" mesh="${yaw_mesh}" cog="${yaw_cog}" mass="${yaw_mass}" >
+    <mesh filename="package://grips_description/meshes/yaw/yaw_collision.dae" />
 		<yaw_inertia />
-	</create_link>
+	</link_collision>
 	<!-- end effector dummy link -->
 	<link name="end_effector" />
 	<!-- camera link -->
-	<create_link name="camera_link" color="black" mesh="${camera_mesh}" cog="${camera_cog}" mass="${camera_mass}" >
+	<link_collision name="camera_link" color="black" mesh="${camera_mesh}" cog="${camera_cog}" mass="${camera_mass}" >
+    <mesh filename="package://grips_description/meshes/camera/camera_collision.dae" />
 		<camera_inertia />
-	</create_link>
+	</link_collision>
 	<!-- Joints -->
 	<joint name="SA" type="revolute">

File: grips_description/urdf/simple_gripper.xacro (robot description, xacro)
@@ -45,10 +45,10 @@
 	</macro>
 	<!-- Meshes -->
-	<property name="gripper_base_mesh" value="package://grips_description/meshes/gripper_base.dae" />
-	<property name="outer_mesh" value="package://grips_description/meshes/outer_pivot.dae" />
-	<property name="r_inner_mesh" value="package://grips_description/meshes/r_inner_pivot.dae" />
-	<property name="l_inner_mesh" value="package://grips_description/meshes/l_inner_pivot.dae" />
-	<property name="r_finger_mesh" value="package://grips_description/meshes/r_finger.dae" />
-	<property name="l_finger_mesh" value="package://grips_description/meshes/l_finger.dae" />
+	<property name="gripper_base_mesh" value="package://grips_description/meshes/gripper/gripper_base.dae" />
+	<property name="outer_mesh" value="package://grips_description/meshes/gripper/outer_pivot.dae" />
+	<property name="r_inner_mesh" value="package://grips_description/meshes/gripper/r_inner_pivot.dae" />
+	<property name="l_inner_mesh" value="package://grips_description/meshes/gripper/l_inner_pivot.dae" />
+	<property name="r_finger_mesh" value="package://grips_description/meshes/gripper/r_finger.dae" />
+	<property name="l_finger_mesh" value="package://grips_description/meshes/gripper/l_finger.dae" />
 	<!-- Joints Dynamics -->
 	<property name="outer_damping" value="0.1" />
