Commit message: Remove namespaces for multi-robot setups because moveit only support planning scenes with only 1 robot

File: grips_description/robots/grips.urdf (robot description, URDF)
Before this commit: robot grips, 11 links, 10 joints
Links:
- removed link camera_link
- removed link coupling_link
- removed link elbow_pivot_link
- removed link forearm_link
- removed link manifold_link
- removed link pitch_link
- removed link upper_arm_link
- removed link yaw_link
- added link camera, mass 0.869; collision mesh filename=package://grips_description/meshes/camera/camera_collision.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; visual mesh filename=package://grips_description/meshes/camera/camera.dae
- added link coupling, mass 0.446; collision mesh filename=package://grips_description/meshes/linkage/coupling.dae; visual mesh filename=package://grips_description/meshes/linkage/coupling.dae
- added link elbow_pivot, mass 0.72; collision mesh filename=package://grips_description/meshes/linkage/elbow_pivot.dae; visual mesh filename=package://grips_description/meshes/linkage/elbow_pivot.dae
- added link forearm, mass 4.935; collision mesh filename=package://grips_description/meshes/forearm/forearm_collisio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; visual mesh filename=package://grips_description/meshes/forearm/forearm.dae
- added link gripper_base, mass 0.923; collision mesh filename=package://grips_description/meshes/gripper/gripper_base.dae; visual mesh filename=package://grips_description/meshes/gripper/gripper_base.dae
- added link l_finger, mass 0.174; collision mesh filename=package://grips_description/meshes/gripper/l_finger.dae; visual mesh filename=package://grips_description/meshes/gripper/l_finger.dae
- added link l_inner, mass 0.194; collision mesh filename=package://grips_description/meshes/gripper/l_inner_pivot.dae; visual mesh filename=package://grips_description/meshes/gripper/l_inner_pivot.dae
- added link l_outer, mass 0.091; collision mesh filename=package://grips_description/meshes/gripper/outer_pivot.dae; visual mesh filename=package://grips_description/meshes/gripper/outer_pivot.dae
- added link manifold, mass 41.111; collision mesh filename=package://grips_description/meshes/manifold/manifold_collis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; visual mesh filename=package://grips_description/meshes/manifold/manifold.dae
- added link pitch, mass 0.679; collision mesh filename=package://grips_description/meshes/pitch/pitch_collision.dae; visual mesh filename=package://grips_description/meshes/pitch/pitch.dae
- added link r_finger, mass 0.174; collision mesh filename=package://grips_description/meshes/gripper/r_finger.dae; visual mesh filename=package://grips_description/meshes/gripper/r_finger.dae
- added link r_inner, mass 0.194; collision mesh filename=package://grips_description/meshes/gripper/r_inner_pivot.dae; visual mesh filename=package://grips_description/meshes/gripper/r_inner_pivot.dae
- added link r_outer, mass 0.091; collision mesh filename=package://grips_description/meshes/gripper/outer_pivot.dae; visual mesh filename=package://grips_description/meshes/gripper/outer_pivot.dae
- added link upper_arm, mass 3.592; collision mesh filename=package://grips_description/meshes/upper_arm/upper_arm_coll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; visual mesh filename=package://grips_description/meshes/upper_arm/upper_arm.dae
- added link yaw, mass 4.689; collision mesh filename=package://grips_description/meshes/yaw/yaw_collision.dae; visual mesh filename=package://grips_description/meshes/yaw/yaw.dae
Joints:
- added joint gripper_anchor: type fixed, parent end_effector, child gripper_base, origin xyz=0 0 0 rpy=0 0 0
- added joint l_finger: type revolute, parent l_inner, child l_finger, origin xyz=0 63.45e-3 0 rpy=0 0 0, axis 0 0 1, limit lower=-1.57079632679 upper=1.57079632679 effort=200 velocity=15
- added joint l_inner: type revolute, parent gripper_base, child l_inner, origin xyz=-31.737e-3 42.19e-3 0 rpy=0 0 0, axis 0 0 1, limit lower=-0.4 upper=1.43 effort=200 velocity=15
- added joint l_outer: type revolute, parent gripper_base, child l_outer, origin xyz=-58.93e-3 26.49e-3 0 rpy=0 0 0, axis 0 0 1, limit lower=-0.4 upper=1.43 effort=200 velocity=15
- added joint r_finger: type revolute, parent r_inner, child r_finger, origin xyz=0 63.45e-3 0 rpy=0 0 0, axis 0 0 1, limit lower=-1.57079632679 upper=1.57079632679 effort=200 velocity=15
- added joint r_inner: type revolute, parent gripper_base, child r_inner, origin xyz=31.737e-3 42.19e-3 0 rpy=0 0 0, axis 0 0 1, limit lower=-1.43 upper=0.4 effort=200 velocity=15
- added joint r_outer: type revolute, parent gripper_base, child r_outer, origin xyz=58.93e-3 26.49e-3 0 rpy=0 0 0, axis 0 0 1, limit lower=-1.43 upper=0.4 effort=200 velocity=15
- joint SA: child manifold_link -> manifold
- joint SE: child upper_arm_link -> upper_arm; parent manifold_link -> manifold
- joint WP: child pitch_link -> pitch; parent forearm_link -> forearm
- joint WR: parent yaw_link -> yaw
- joint WY: child yaw_link -> yaw; parent pitch_link -> pitch
- joint camera_joint: child camera_link -> camera; parent yaw_link -> yaw
- joint linkage_bl: child elbow_pivot_link -> elbow_pivot; parent coupling_link -> coupling
- joint linkage_tl: child coupling_link -> coupling; parent forearm_link -> forearm
- joint linkage_tr: child forearm_link -> forearm; parent upper_arm_link -> upper_arm

File: grips_description/robots/grips.xacro (robot description, xacro)
@@ -1,4 +1,4 @@
 <?xml version="1.0"?>
-<robot name="grips_simple_gripper" xmlns:xacro="http://www.ros.org/wiki/xacro">
+<robot name="grips" xmlns:xacro="http://www.ros.org/wiki/xacro">
 	<!-- Import common macros-->
 	<xacro:include filename="$(find grips_description)/urdf/common.xacro" />
@@ -6,7 +6,11 @@
 	<xacro:include filename="$(find grips_description)/urdf/materials.xacro" />
 	<!-- Import robot without gripper -->
-	<xacro:include filename="$(find grips_description)/urdf/grips.xacro" />
+	<xacro:include filename="$(find grips_description)/urdf/grips_macro.xacro" />
 	<!-- Import simple gripper -->
-	<xacro:include filename="$(find grips_description)/urdf/simple_gripper.xacro" />
+	<xacro:include filename="$(find grips_description)/urdf/simple_gripper_macro.xacro" />
+  <!-- Create the grips robot -->
+  <grips_robot name=""/>
+  <!-- Create the simple_gripper -->
+  <simple_gripper name=""/>
 	<!-- Used for fixing robot to Gazebo 'base_link' -->
 	<link name="world" />
@@ -16,5 +20,5 @@
 		<child link="base_link" />
 	</joint>
-	<!-- Used for fixing the gripper to the robot -->
+  <!-- Used for fixing the gripper to the robot -->
 	<joint name="gripper_anchor" type="fixed">
 		<origin xyz="0 0 0" rpy="0 0 0" />
@@ -25,8 +29,4 @@
 	<gazebo>
 		<plugin name="ros_control" filename="libgazebo_ros_control.so">
-<!--
-			<robotNamespace>/grips_simple_gripper</robotNamespace>
-      <robotParam>/grips_simple_gripper/robot_description</robotParam>
--->
 		</plugin>
 	</gazebo>

File: grips_description/urdf/common.xacro (robot description, xacro)
@@ -1,5 +1,147 @@
 <?xml version="1.0"?>
 <robot xmlns:xacro="http://www.ros.org/wiki/xacro">
-	<!-- Link's Macro -->
+  <!-- Auxiliar Values -->
+	<property name="pi" value="3.1415926535897931" />
+	<property name="gripper_effort" value="200" />
+	<property name="gripper_velocity" value="15" />
+  <!-- Auxiliar Values -->
+	<property name="pi" value="3.1415926535897931" />
+	<property name="max_effort" value="200" />
+  <property name="max_velocity" value="15" />
+	<!-- Links Mass -->
+	<property name="base_mass" value="1.208" />
+	<property name="manifold_mass" value="41.111" />
+	<property name="upper_arm_mass" value="3.592" />
+	<property name="elbow_pivot_mass" value="0.72" />
+	<property name="coupling_mass" value="0.446" />
+	<property name="forearm_mass" value="4.935" />
+	<property name="pitch_mass" value="0.679" />
+	<property name="yaw_mass" value="4.689" />
+	<property name="camera_mass" value="0.869" />
+	<!-- Links COG -->
+	<property name="base_cog" value="0 0 7e-3" />
+	<property name="manifold_cog" value="0 2e-3 0.21" />
+	<property name="upper_arm_cog" value="0 5e-3 0.227" />
+	<property name="elbow_pivot_cog" value="-3.6e-10 80.686e-3 -6.33e-5" />
+	<property name="coupling_cog" value="0 0 -0.26035" />
+	<property name="forearm_cog" value="0 0.155337 0.012119" />
+	<property name="pitch_cog" value="0 0.065 0" />
+	<property name="yaw_cog" value="-1e-3 95.791e-3 18.273e-3" />
+	<property name="camera_cog" value="0.077 0.007 0.002" />
+	<!-- Links Inertia -->
+	<macro name="base_inertia">
+		<inertia ixx="0.003" ixy="0.0" ixz="0.0" iyy="0.003" iyz="0.0"
+			izz="0.006" />
+	</macro>
+	<macro name="manifold_inertia">
+		<inertia 	ixx="0.549" 	ixy="-9.556e-5"		ixz="-5.871e-5"
+							iyy="0.855"	iyz="2e-3"
+							izz="0.605" />
+	</macro>
+	<macro name="upper_arm_inertia">
+		<inertia 	ixx="0.103" ixy="0" ixz="0"
+							iyy="0.106" iyz="0.004"
+							izz="0.013" />
+	</macro>
+	<macro name="elbow_pivot_inertia">
+		<inertia 	ixx="0.002" ixy="-3.231e-27" ixz="0"
+							iyy="3.397e-4" iyz="-1.919e-5"
+							izz="0.002" />
+	</macro>
+	<macro name="coupling_inertia">
+		<inertia 	ixx="0.011" ixy="-3.231e-27" ixz="0"
+							iyy="0.011" iyz="0"
+							izz="2.102e-5" />
+	</macro>
+	<macro name="forearm_inertia">
+		<inertia 	ixx="0.073" ixy="0" ixz="0"
+							iyy="0.009" iyz="0.004"
+							izz="0.073" />
+	</macro>
+	<macro name="pitch_inertia">
+		<inertia 	ixx="0.003" ixy="0" ixz="0"
+							iyy="0.002" iyz="0.004"
+							izz="0.002" />
+	</macro>
+	<macro name="yaw_inertia">
+		<inertia 	ixx="0.027" ixy="1.597e-4" ixz="-2.174e-4"
+							iyy="0.009" iyz="-0.003"
+							izz="0.026" />
+	</macro>
+	<macro name="camera_inertia">
+		<inertia 	ixx="0.001" ixy="-1.561e-4" ixz="-5.859e-5"
+							iyy="0.002" iyz="3.295e-5"
+							izz="0.002" />
+	</macro>
+	<!-- Meshes -->
+	<property name="base_mesh" value="package://grips_description/meshes/base/base.dae" />
+	<property name="manifold_mesh" value="package://grips_description/meshes/manifold/manifold.dae" />
+	<property name="upper_arm_mesh" value="package://grips_description/meshes/upper_arm/upper_arm.dae" />
+	<property name="elbow_pivot_mesh" value="package://grips_description/meshes/linkage/elbow_pivot.dae" />
+	<property name="coupling_mesh" value="package://grips_description/meshes/linkage/coupling.dae" />
+	<property name="forearm_mesh" value="package://grips_description/meshes/forearm/forearm.dae" />
+	<property name="pitch_mesh" value="package://grips_description/meshes/pitch/pitch.dae" />
+	<property name="yaw_mesh" value="package://grips_description/meshes/yaw/yaw.dae" />
+	<property name="camera_mesh" value="package://grips_description/meshes/camera/camera.dae" />
+	<!-- Joints Dynamics -->
+	<property name="SA_damping" value="5" />
+	<property name="SE_damping" value="5" />
+	<property name="linkage_damping" value="0.5" />
+	<property name="linkage_friction" value="0.5" />
+	<property name="WP_damping" value="5" />
+	<property name="WY_damping" value="5" />
+	<property name="WR_damping" value="0.5" />
+	<!-- Links Mass -->
+	<property name="gripper_base_mass" value="0.923" />
+	<property name="outer_mass" value="0.091" />
+	<property name="inner_mass" value="0.194" />
+	<property name="finger_mass" value="0.174" />
+	<!-- Links COG -->
+	<property name="gripper_base_cog" value="0 26.28e-3 0" />
+	<property name="outer_cog" value="0 31.725e-3 0" />
+	<property name="r_inner_cog" value="-0.316e-3 23.873e-3 0" />
+	<property name="l_inner_cog" value="0.316e-3 23.873e-3 0" />
+	<property name="r_finger_cog" value="3.441e-3 20.353e-3 0" />
+	<property name="l_finger_cog" value="-3.441e-3 20.353e-3 0" />
+	<!-- Links Inertia -->
+	<macro name="gripper_base_inertia">
+		<inertia ixx="9.67e-4" ixy="0.0" ixz="0.0" iyy="0.002" iyz="0.0"
+			izz="0.002" />
+	</macro>
+	<macro name="outer_inertia">
+		<inertia ixx="4.664e-5" ixy="0.0" ixz="0.0" iyy="5.519e-6"
+			iyz="0.0" izz="4.682e-5" />
+	</macro>
+	<macro name="r_inner_inertia">
+		<inertia ixx="1.179e-4" ixy="1.347e-6" ixz="0.0" iyy="5.647e-5"
+			iyz="0.0" izz="7.353e-5" />
+	</macro>
+	<macro name="l_inner_inertia">
+		<inertia ixx="1.179e-4" ixy="-1.347e-6" ixz="0.0" iyy="5.647e-5"
+			iyz="0.0" izz="7.353e-5" />
+	</macro>
+	<macro name="r_finger_inertia">
+		<inertia ixx="1.65e-4" ixy="3.16e-5" ixz="0.0" iyy="3.595e-5"
+			iyz="0.0" izz="1.701e-4" />
+	</macro>
+	<macro name="l_finger_inertia">
+		<inertia ixx="1.65e-4" ixy="-3.16e-5" ixz="0.0" iyy="3.595e-5"
+			iyz="0.0" izz="1.701e-4" />
+	</macro>
+	<!-- Meshes -->
+	<property name="gripper_base_mesh" value="package://grips_description/meshes/gripper/gripper_base.dae" />
+	<property name="outer_mesh" value="package://grips_description/meshes/gripper/outer_pivot.dae" />
+	<property name="r_inner_mesh" value="package://grips_description/meshes/gripper/r_inner_pivot.dae" />
+	<property name="l_inner_mesh" value="package://grips_description/meshes/gripper/l_inner_pivot.dae" />
+	<property name="r_finger_mesh" value="package://grips_description/meshes/gripper/r_finger.dae" />
+	<property name="l_finger_mesh" value="package://grips_description/meshes/gripper/l_finger.dae" />
+	<!-- Joints Dynamics -->
+	<property name="outer_damping" value="0.1" />
+	<property name="inner_damping" value="0.1" />
+	<property name="finger_damping" value="0.1" />
+	<property name="inner_friction" value="0" />
+	<property name="outer_friction" value="0" />
+	<property name="finger_friction" value="0" />
+	<!-- Link's Macros -->
 	<macro name="create_link" params="name color mesh mass cog *inertia">
 		<link name="${name}">
