Commit message: Added custom ft_sensor. Depends on this https://github.com/ros-simulation/gazebo_ros_pkgs/pull/204

File: grips_description/robots/grips_robotiq.urdf (robot description, URDF)
Before this commit: robot grips, 13 links, 12 joints
Links:
- added link finger_1_link_0, mass 0.05; collision mesh filename=package://robotiq_s_model_visualization/meshes/s-model_arti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; visual mesh filename=package://robotiq_s_model_visualization/meshes/s-model_arti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
- added link finger_1_link_1, mass 0.15; collision mesh filename=package://robotiq_s_model_visualization/meshes/s-model_arti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; visual mesh filename=package://robotiq_s_model_visualization/meshes/s-model_arti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
- added link finger_1_link_2, mass 0.15; collision mesh filename=package://robotiq_s_model_visualization/meshes/s-model_arti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; visual mesh filename=package://robotiq_s_model_visualization/meshes/s-model_arti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
- added link finger_1_link_3, mass 0.05; collision mesh filename=package://robotiq_s_model_visualization/meshes/s-model_arti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; visual mesh filename=package://robotiq_s_model_visualization/meshes/s-model_arti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
- added link finger_2_link_0, mass 0.05; collision mesh filename=package://robotiq_s_model_visualization/meshes/s-model_arti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; visual mesh filename=package://robotiq_s_model_visualization/meshes/s-model_arti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
- added link finger_2_link_1, mass 0.15; collision mesh filename=package://robotiq_s_model_visualization/meshes/s-model_arti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; visual mesh filename=package://robotiq_s_model_visualization/meshes/s-model_arti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
- added link finger_2_link_2, mass 0.15; collision mesh filename=package://robotiq_s_model_visualization/meshes/s-model_arti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; visual mesh filename=package://robotiq_s_model_visualization/meshes/s-model_arti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
- added link finger_2_link_3, mass 0.05; collision mesh filename=package://robotiq_s_model_visualization/meshes/s-model_arti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; visual mesh filename=package://robotiq_s_model_visualization/meshes/s-model_arti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
- added link finger_middle_link_0, mass 0.05; collision mesh filename=package://robotiq_s_model_visualization/meshes/s-model_arti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; visual mesh filename=package://robotiq_s_model_visualization/meshes/s-model_arti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
- added link finger_middle_link_1, mass 0.15; collision mesh filename=package://robotiq_s_model_visualization/meshes/s-model_arti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; visual mesh filename=package://robotiq_s_model_visualization/meshes/s-model_arti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
- added link finger_middle_link_2, mass 0.15; collision mesh filename=package://robotiq_s_model_visualization/meshes/s-model_arti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; visual mesh filename=package://robotiq_s_model_visualization/meshes/s-model_arti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
- added link finger_middle_link_3, mass 0.05; collision mesh filename=package://robotiq_s_model_visualization/meshes/s-model_arti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; visual mesh filename=package://robotiq_s_model_visualization/meshes/s-model_arti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
- added link ft_end_effector
- added link ft_robotiq_plate, mass 0.2304; collision mesh filename=package://grips_description/meshes/visual/ft_robotiq_plate.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; visual mesh filename=package://grips_description/meshes/visual/ft_robotiq_plate.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
- added link ft_sensor, mass 0.2396; collision mesh filename=package://grips_description/meshes/visual/ft_sensor.dae; visual mesh filename=package://grips_description/meshes/visual/ft_sensor.dae
- added link palm; collision mesh filename=package://robotiq_s_model_visualization/meshes/s-model_arti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; visual mesh filename=package://robotiq_s_model_visualization/meshes/s-model_arti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
Joints:
- added joint finger_1_joint_1: type revolute, parent finger_1_link_0, child finger_1_link_1, origin xyz=0.020 0 0 rpy=0 0 0, axis 0 0 1, limit lower=0 upper=3.1416 effort=100 velocity=100
- added joint finger_1_joint_2: type revolute, parent finger_1_link_1, child finger_1_link_2, origin xyz=0.050 -.028 0 rpy=0 0 -0.52, axis 0 0 1, limit lower=0 upper=3.1416 effort=100 velocity=100
- added joint finger_1_joint_3: type revolute, parent finger_1_link_2, child finger_1_link_3, origin xyz=0.039 0 0 rpy=0 0 0, axis 0 0 1, limit lower=0 upper=3.1416 effort=100 velocity=100
- added joint finger_2_joint_1: type revolute, parent finger_2_link_0, child finger_2_link_1, origin xyz=0.020 0 0 rpy=0 0 0, axis 0 0 1, limit lower=0 upper=3.1416 effort=100 velocity=100
- added joint finger_2_joint_2: type revolute, parent finger_2_link_1, child finger_2_link_2, origin xyz=0.050 -.028 0 rpy=0 0 -0.52, axis 0 0 1, limit lower=0 upper=3.1416 effort=100 velocity=100
- added joint finger_2_joint_3: type revolute, parent finger_2_link_2, child finger_2_link_3, origin xyz=0.039 0 0 rpy=0 0 0, axis 0 0 1, limit lower=0 upper=3.1416 effort=100 velocity=100
- added joint finger_middle_joint_1: type revolute, parent finger_middle_link_0, child finger_middle_link_1, origin xyz=0.020 0 0 rpy=0 0 0, axis 0 0 1, limit lower=0 upper=3.1416 effort=100 velocity=100
- added joint finger_middle_joint_2: type revolute, parent finger_middle_link_1, child finger_middle_link_2, origin xyz=0.050 -.028 0 rpy=0 0 -0.52, axis 0 0 1, limit lower=0 upper=3.1416 effort=100 velocity=100
- added joint finger_middle_joint_3: type revolute, parent finger_middle_link_2, child finger_middle_link_3, origin xyz=0.039 0 0 rpy=0 0 0, axis 0 0 1, limit lower=0 upper=3.1416 effort=100 velocity=100
- added joint ft_end_joint: type fixed, parent ft_robotiq_plate, child ft_end_effector, origin xyz=0 0 0 rpy=-1.57079632679 0 0
- added joint ft_plate_joint: type fixed, parent ft_sensor, child ft_robotiq_plate, origin xyz=0 -11e-3 0 rpy=-1.57079632679 0 0
- added joint ft_sensor_joint: type fixed, parent ft_wrist_plate, child ft_sensor, origin xyz=0 0 0.0564 rpy=-1.57079632679 0 0
- added joint palm_finger_1_joint: type revolute, parent palm, child finger_1_link_0, origin xyz=-0.0455 0.0214 0.036 rpy=0 3.1416 -1.57, axis 0 1 0, limit lower=-0.16 upper=0.25 effort=100 velocity=100
- added joint palm_finger_2_joint: type revolute, parent palm, child finger_2_link_0, origin xyz=-0.0455 0.0214 -0.036 rpy=0 3.1416 -1.57, axis 0 1 0, limit lower=-0.25 upper=0.16 effort=100 velocity=100
- added joint palm_finger_middle_joint: type fixed, parent palm, child finger_middle_link_0, origin xyz=0.0455 0.0214 0 rpy=0 0 1.57, axis 0 0 1
- added joint robotiq_anchor: type fixed, parent ft_end_effector, child palm, origin xyz=0 54e-3 0 rpy=0 0 0
- joint ft_wrist_joint: origin xyz=0 4.7e-3 0 rpy=$0 0 0 -> xyz=0 0 0 rpy=0 0 0

File: grips_description/robots/grips_robotiq.xacro (robot description, xacro)
@@ -22,7 +22,27 @@
   </joint>
   <!-- Add the ft_sensor -->
-  <ftsensor name="${robot_name}" parent="end_effector"/>
+  <ftsensor name="${robot_name}" parent="${robot_name}end_effector"/>
+  <gazebo reference="${robot_name}WR">
+    <provideFeedback>true</provideFeedback>
+    <!-- FIXME: This sensor tag is never included in the sdf -->
+    <sensor type="force_torque" name="${robot_name}force_torque_sensor">
+      <always_on>1</always_on>
+      <update_rate>100.0</update_rate>
+      <visualize>1</visualize>
+      <force_torque name="${robot_name}ft_sensor">
+        <frame>child</frame>
+      </force_torque>
+    </sensor>
+    <!-- *************************************************** -->
+  </gazebo>
+  <gazebo>
+    <plugin name="ft_sensor" filename="libgazebo_ros_ft_sensor.so">
+      <updateRate>100.0</updateRate>
+      <topicName>ft_sensor</topicName>
+      <jointName>${robot_name}WR</jointName>
+    </plugin>
+  </gazebo>
    Add robotiq hand
-  <s-model_articulated prefix=""/>
+  <s-model_articulated prefix="${robot_name}"/>
   <!-- Used for fixing Robotiq to the FT sensor -->
   <joint name="robotiq_anchor" type="fixed">

File: grips_description/urdf/ftsensor.xacro (robot description, xacro)
@@ -76,4 +76,32 @@
       <child link="${name}ft_end_effector" />
     </joint>
+<!--
+    <gazebo reference="${name}ft_plate_joint">
+      <physics>
+        <provide_feedback>1</provide_feedback>
+      </physics>
+      <sensor type="force_torque" name="${name}force_torque_sensor">
+        <always_on>1</always_on>
+        <update_rate>1000.0</update_rate>
+        <visualize>1</visualize>
+        <force_torque name="${name}force_torque_sensor">
+          <frame>${name}ft_robotiq_plate</frame>
+        </force_torque>
+        <plugin name="ft_sensor_plugin" filename="libgazebo_ros_ft_sensor.so">
+          <alwaysOn>1</alwaysOn>
+          <updateRate>1000.0</updateRate>
+          <robotNamespace>grips_robotiq</robotNamespace>
+          <topicName>ft_sensor</topicName>
+        </plugin>
+      </sensor>
+    </gazebo>
+    <transmission name="${name}ft_plate_joint_tran">
+      <type>hardware_interface/ForceTorqueSensorInterface</type>
+      <joint name="${name}ft_plate_joint" />
+      <actuator name="${name}ft_plate_joint_motor">
+        <hardwareInterface>EffortJointInterface</hardwareInterface>
+        <mechanicalReduction>1</mechanicalReduction>
+      </actuator>
+    </transmission>-->
   </macro>
 </robot>

Commit message: Minor changes

File: grips_description/robots/grips_robotiq.urdf (robot description, URDF)
Before this commit: robot grips, 29 links, 28 joints
Links:
- added link imu_board, mass 0.059; collision box size=0.06477 0.06604 0.00337; visual box size=0.06477 0.06604 0.00337
- added link imu_sensor, mass 0.0245; collision mesh filename=package://grips_description/meshes/visual/adis1640x.dae; visual mesh filename=package://grips_description/meshes/visual/adis1640x.dae
Joints:
- added joint board_joint: type fixed, parent end_effector, child imu_board, origin xyz=0 0.13 0.067005 rpy=0 0 -1.57079632679
- added joint imu_joint: type fixed, parent imu_board, child imu_sensor, origin xyz=0 0 0.002435 rpy=0 0 0

File: grips_description/urdf/ft_sensor.xacro (robot description, xacro)
@@ -94,5 +94,5 @@
         <robotNamespace>/grips_robotiq</robotNamespace>
         <updateRate>100.0</updateRate>
-        <topicName>ft_sensor</topicName>
+        <topicName>ft_raw</topicName>
         <jointName>${name}WR</jointName>
       </plugin>

File: grips_description/urdf/imu_sensor.xacro (robot description, xacro)
@@ -63,6 +63,6 @@
       <plugin name="imu_sensor" filename="libgazebo_ros_imu.so">
         <robotNamespace>/grips_robotiq</robotNamespace>
-        <updateRate>100.0</updateRate>
-        <topicName>imu_sensor</topicName>
+        <updateRate>500.0</updateRate>
+        <topicName>imu</topicName>
         <bodyName>${prefix}imu_board</bodyName>
       </plugin>
