Commit message: Added grips_robotiq description. It's working in gazebo

File: grips_description/robots/grips_robotiq.xacro (robot description, xacro)
@@ -7,6 +7,8 @@
   <!-- Import robot without gripper -->
   <xacro:include filename="$(find grips_description)/urdf/grips_macro.xacro" />
-  <!-- Import simple gripper -->
+  <!-- Import ft sensor -->
   <xacro:include filename="$(find grips_description)/urdf/ftsensor.xacro" />
+  <!-- Import robotiq s model -->
+  <xacro:include filename="$(find robotiq_s_model_visualization)/cfg/s-model_articulated_macro.xacro" />
   <property name="robot_name" value="" />
   <!-- Create the grips robot -->
@@ -21,8 +23,16 @@
   <!-- Add the ft_sensor -->
   <ftsensor name="${robot_name}" parent="end_effector"/>
+   Add robotiq hand
+  <s-model_articulated prefix=""/>
+  <!-- Used for fixing Robotiq to the FT sensor -->
+  <joint name="robotiq_anchor" type="fixed">
+    <origin xyz="0 54e-3 0" rpy="0 0 0" />
+    <parent link="ft_end_effector" />
+    <child link="palm" />
+  </joint>
   <!-- ros_control plugin -->
   <gazebo>
     <plugin name="ros_control" filename="libgazebo_ros_control.so">
-      <robotNamespace>/grips</robotNamespace>
+      <robotNamespace>/grips_robotiq</robotNamespace>
     </plugin>
   </gazebo>

Commit message: grips_description: Added IMU sensor to the grips_robotiq robot

File: grips_description/robots/grips_robotiq.xacro (robot description, xacro)
@@ -8,5 +8,7 @@
   <xacro:include filename="$(find grips_description)/urdf/grips_macro.xacro" />
   <!-- Import ft sensor -->
-  <xacro:include filename="$(find grips_description)/urdf/ftsensor.xacro" />
+  <xacro:include filename="$(find grips_description)/urdf/ft_sensor.xacro" />
+  <!-- Import imu sensor -->
+  <xacro:include filename="$(find grips_description)/urdf/imu_sensor.xacro" />
   <!-- Import robotiq s model -->
   <xacro:include filename="$(find robotiq_s_model_visualization)/cfg/s-model_articulated_macro.xacro" />
@@ -14,4 +16,16 @@
   <!-- Create the grips robot -->
   <grips_robot name="${robot_name}"/>
+  <!-- Add the ft_sensor -->
+  <ft_sensor name="${robot_name}" parent="${robot_name}end_effector"/>
+  <!-- Add the imu_sensor -->
+  <imu_sensor prefix="${robot_name}" parent="${robot_name}end_effector">
+    <origin xyz="0 0.13 ${board_z_size+63.635e-3}" rpy="0 0 ${-pi/2}" />
+  </imu_sensor>
+  <!-- Add robotiq hand -->
+  <s-model_articulated prefix="${robot_name}"/>
+  <gazebo reference="${robot_name}palm">
+    <material>Gazebo/FlatBlack</material>
+    <turnGravityOff>false</turnGravityOff>
+  </gazebo>
   <!-- Used for fixing robot to Gazebo 'base_link' -->
   <link name="world" />
@@ -21,33 +35,9 @@
     <child link="base_link" />
   </joint>
-  <!-- Add the ft_sensor -->
-  <ftsensor name="${robot_name}" parent="${robot_name}end_effector"/>
-  <gazebo reference="${robot_name}WR">
-    <provideFeedback>true</provideFeedback>
-    <!-- FIXME: This sensor tag is never included in the sdf -->
-    <sensor type="force_torque" name="${robot_name}force_torque_sensor">
-      <always_on>1</always_on>
-      <update_rate>100.0</update_rate>
-      <visualize>1</visualize>
-      <force_torque name="${robot_name}ft_sensor">
-        <frame>child</frame>
-      </force_torque>
-    </sensor>
-    <!-- *************************************************** -->
-  </gazebo>
-  <gazebo>
-    <plugin name="ft_sensor" filename="libgazebo_ros_ft_sensor.so">
-      <updateRate>100.0</updateRate>
-      <topicName>ft_sensor</topicName>
-      <jointName>${robot_name}WR</jointName>
-    </plugin>
-  </gazebo>
-   Add robotiq hand
-  <s-model_articulated prefix="${robot_name}"/>
   <!-- Used for fixing Robotiq to the FT sensor -->
   <joint name="robotiq_anchor" type="fixed">
     <origin xyz="0 54e-3 0" rpy="0 0 0" />
-    <parent link="ft_end_effector" />
-    <child link="palm" />
+    <parent link="${robot_name}ft_end_effector" />
+    <child link="${robot_name}palm" />
   </joint>
   <!-- ros_control plugin -->

File: grips_description/urdf/common.xacro (robot description, xacro)
@@ -195,3 +195,9 @@
     </transmission>
   </macro>
+  <!--Inertial macro for a box. Units are kg*m^2-->
+  <macro name="box_inertia" params="m x y z">
+    <inertia  ixx="${m*(y*y+z*z)/12}" ixy = "0" ixz = "0"
+              iyy="${m*(x*x+z*z)/12}" iyz = "0"
+              izz="${m*(x*x+z*z)/12}" />
+  </macro>
 </robot>

File: grips_description/urdf/ft_sensor.xacro (robot description, xacro)
@@ -34,5 +34,5 @@
               ixy="0.0"       ixz="0.0"       iyz="0.0" />
   </macro>
-  <macro name="ftsensor" params="name parent">
+  <macro name="ft_sensor" params="name parent">
     <!-- Links -->
     <create_link name="${name}ft_kraft_plate" color="black" mesh="${ft_kraft_plate_mesh}" mass="${ft_kraft_plate_mass}" cog="${ft_kraft_plate_cog}" >
@@ -76,32 +76,26 @@
       <child link="${name}ft_end_effector" />
     </joint>
-<!--
-    <gazebo reference="${name}ft_plate_joint">
-      <physics>
-        <provide_feedback>1</provide_feedback>
-      </physics>
+    <gazebo reference="${name}WR">
+      <provideFeedback>true</provideFeedback>
+      <!-- FIXME: This sensor tag is never included in the sdf -->
       <sensor type="force_torque" name="${name}force_torque_sensor">
         <always_on>1</always_on>
-        <update_rate>1000.0</update_rate>
+        <update_rate>100.0</update_rate>
         <visualize>1</visualize>
-        <force_torque name="${name}force_torque_sensor">
-          <frame>${name}ft_robotiq_plate</frame>
+        <force_torque name="${name}ft_sensor">
+          <frame>child</frame>
         </force_torque>
-        <plugin name="ft_sensor_plugin" filename="libgazebo_ros_ft_sensor.so">
-          <alwaysOn>1</alwaysOn>
-          <updateRate>1000.0</updateRate>
-          <robotNamespace>grips_robotiq</robotNamespace>
-          <topicName>ft_sensor</topicName>
-        </plugin>
       </sensor>
+      <!-- *************************************************** -->
     </gazebo>
-    <transmission name="${name}ft_plate_joint_tran">
-      <type>hardware_interface/ForceTorqueSensorInterface</type>
-      <joint name="${name}ft_plate_joint" />
-      <actuator name="${name}ft_plate_joint_motor">
-        <hardwareInterface>EffortJointInterface</hardwareInterface>
-        <mechanicalReduction>1</mechanicalReduction>
-      </actuator>
-    </transmission>-->
+    <!-- FT Sensor Plugin -->
+    <gazebo>
+      <plugin name="ft_sensor" filename="libgazebo_ros_ft_sensor.so">
+        <robotNamespace>/grips_robotiq</robotNamespace>
+        <updateRate>100.0</updateRate>
+        <topicName>ft_sensor</topicName>
+        <jointName>${name}WR</jointName>
+      </plugin>
+    </gazebo>
   </macro>
 </robot>

File: grips_description/urdf/materials.xacro (robot description, xacro)
@@ -1,30 +1,30 @@
 <?xml version="1.0"?>
 <robot>
-	<material name="black">
-		<color rgba="0.0 0.0 0.0 1.0" />
-	</material>
-	<material name="blue">
-		<color rgba="0.0 0.0 0.8 1.0" />
-	</material>
-	<material name="green">
-		<color rgba="0.0 0.8 0.0 1.0" />
-	</material>
-	<material name="grey">
-		<color rgba="0.2 0.2 0.2 1.0" />
-	</material>
-	<material name="orange">
-		<color rgba="${255/255} ${108/255} ${10/255} 1.0" />
-	</material>
-	<material name="brown">
-		<color rgba="${222/255} ${207/255} ${195/255} 1.0" />
-	</material>
-	<material name="red">
-		<color rgba="0.8 0.0 0.0 1.0" />
-	</material>
-	<material name="white">
-		<color rgba="1.0 1.0 1.0 1.0" />
-	</material>
-	<material name="metal_seamed">
-		<color rgba="0.4627450980392157 0.4666666666666667 0.4509803921568628 1.0" />
-	</material>
+  <material name="black">
+    <color rgba="0.0 0.0 0.0 1.0" />
+  </material>
+  <material name="blue">
+    <color rgba="0.0 0.0 0.8 1.0" />
+  </material>
+  <material name="green">
+    <color rgba="0.0 0.8 0.0 1.0" />
+  </material>
+  <material name="grey">
+    <color rgba="0.2 0.2 0.2 1.0" />
+  </material>
+  <material name="orange">
+    <color rgba="${255/255} ${108/255} ${10/255} 1.0" />
+  </material>
+  <material name="brown">
+    <color rgba="${222/255} ${207/255} ${195/255} 1.0" />
+  </material>
+  <material name="red">
+    <color rgba="0.8 0.0 0.0 1.0" />
+  </material>
+  <material name="white">
+    <color rgba="1.0 1.0 1.0 1.0" />
+  </material>
+  <material name="metal_seamed">
+    <color rgba="0.4627450980392157 0.4666666666666667 0.4509803921568628 1.0" />
+  </material>
 </robot>

Commit message: Simplified grips and robotiq models for sake of sanity

File: grips_description/robots/grips_robotiq.xacro (robot description, xacro)
@@ -12,5 +12,5 @@
   <xacro:include filename="$(find grips_description)/urdf/imu_sensor.xacro" />
   <!-- Import robotiq s model -->
-  <xacro:include filename="$(find robotiq_s_model_visualization)/cfg/s-model_articulated_macro.xacro" />
+  <xacro:include filename="$(find robotiq_s_model_visualization)/cfg/s-model_fixed_macro.xacro" />
   <property name="robot_name" value="" />
   <!-- Create the grips robot -->
@@ -23,5 +23,5 @@
   </imu_sensor>
   <!-- Add robotiq hand -->
-  <s-model_articulated prefix="${robot_name}"/>
+  <s-model_fixed prefix="${robot_name}"/>
   <gazebo reference="${robot_name}palm">
     <material>Gazebo/FlatBlack</material>

File: grips_description/urdf/grips_macro.xacro (robot description, xacro)
@@ -17,12 +17,4 @@
       <upper_arm_inertia />
     </link_collision>
-    <!-- elbow pivot link -->
-    <create_link name="${name}elbow_pivot" color="black" mesh="${elbow_pivot_mesh}" cog="${elbow_pivot_cog}" mass="${elbow_pivot_mass}" >
-      <elbow_pivot_inertia />
-    </create_link>
-    <!-- coupling link -->
-    <create_link name="${name}coupling" color="black" mesh="${coupling_mesh}" cog="${coupling_cog}" mass="${coupling_mass}" >
-      <coupling_inertia />
-    </create_link>
     <!-- forearm link -->
     <link_collision name="${name}forearm" color="black" mesh="${forearm_mesh}" cog="${forearm_cog}" mass="${forearm_mass}" >
@@ -102,21 +94,4 @@
       <origin xyz="0 ${0.190892/2} 0.25" rpy="0 ${pi/6} ${pi/2}"/>
     </joint>
-    <!-- four-bar linkage -->
-    <joint name="${name}linkage_tl" type="continuous">
-      <child link="${name}coupling" />
-      <parent link="${name}forearm" />
-      <axis xyz="1 0 0" />
-      <origin xyz="0 -0.123444 0.029845" rpy="0.019320795 0 0" />
-      <limit effort="${max_effort}" velocity="${max_velocity}" />
-      <dynamics damping="${linkage_damping}" friction="${linkage_friction}"/>
-    </joint>
-    <joint name="${name}linkage_bl" type="continuous">
-      <child link="${name}elbow_pivot" />
-      <parent link="${name}coupling" />
-      <axis xyz="1 0 0" />
-      <origin xyz="0 0 -0.5207" rpy="-0.24521876 0 0" />
-      <limit effort="${max_effort}" velocity="${max_velocity}" />
-      <dynamics damping="${linkage_damping}" friction="${linkage_friction}"/>
-    </joint>
     <!-- Transmissions -->
     <simple_transmission joint="${name}SA" />
@@ -126,6 +101,4 @@
     <simple_transmission joint="${name}WR" />
     <simple_transmission joint="${name}linkage_tr" />
-    <simple_transmission joint="${name}linkage_tl" />
-    <simple_transmission joint="${name}linkage_bl" />
     <gazebo reference="${name}base_link">
       <material>Telerobcar/MetalSeamed</material>
@@ -137,12 +110,4 @@
     </gazebo>
     <gazebo reference="${name}upper_arm">
-      <material>Telerobcar/MetalSeamed</material>
-      <selfCollide>false</selfCollide>
-    </gazebo>
-    <gazebo reference="${name}elbow_pivot">
-      <material>Telerobcar/MetalSeamed</material>
-      <selfCollide>false</selfCollide>
-    </gazebo>
-    <gazebo reference="${name}coupling">
       <material>Telerobcar/MetalSeamed</material>
       <selfCollide>false</selfCollide>
