Commit message: Added labview_server.py node to control the real grips slave

File: grips_description/robots/bimanual.urdf (robot description, URDF)
Before this commit: robot grips, 35 links, 34 joints
Joints:
- joint left_SA: limit lower=-1.57079632679 upper=1.57079632679 effort=200 velocity=15 -> lower=-1.57079632679 upper=1.57079632679 effort=200 velocity=10
- joint left_SE: limit lower=-1.57079632679 upper=0.523598775598 effort=200 velocity=15 -> lower=-1.57079632679 upper=0.523598775598 effort=200 velocity=10
- joint left_WP: limit lower=-1.1 upper=0.581 effort=200 velocity=15 -> lower=-1.1 upper=0.581 effort=200 velocity=10
- joint left_WY: limit lower=-1.01 upper=0.675 effort=200 velocity=15 -> lower=-1.01 upper=0.675 effort=200 velocity=10
- joint left_linkage_bl: limit effort=200 velocity=15 -> effort=200 velocity=10
- joint left_linkage_tl: limit effort=200 velocity=15 -> effort=200 velocity=10
- joint left_linkage_tr: limit lower=-1.28 upper=1.0471975512 effort=200 velocity=15 -> lower=-1.28 upper=1.0471975512 effort=200 velocity=10
- joint right_SA: limit lower=-1.57079632679 upper=1.57079632679 effort=200 velocity=15 -> lower=-1.57079632679 upper=1.57079632679 effort=200 velocity=10
- joint right_SE: limit lower=-1.57079632679 upper=0.523598775598 effort=200 velocity=15 -> lower=-1.57079632679 upper=0.523598775598 effort=200 velocity=10
- joint right_WP: limit lower=-1.1 upper=0.581 effort=200 velocity=15 -> lower=-1.1 upper=0.581 effort=200 velocity=10
- joint right_WY: limit lower=-1.01 upper=0.675 effort=200 velocity=15 -> lower=-1.01 upper=0.675 effort=200 velocity=10
- joint right_linkage_bl: limit effort=200 velocity=15 -> effort=200 velocity=10
- joint right_linkage_tl: limit effort=200 velocity=15 -> effort=200 velocity=10
- joint right_linkage_tr: limit lower=-1.28 upper=1.0471975512 effort=200 velocity=15 -> lower=-1.28 upper=1.0471975512 effort=200 velocity=10

File: grips_description/robots/grips.urdf (robot description, URDF)
Before this commit: robot grips, 18 links, 17 joints
Joints:
- joint SA: limit lower=-1.57079632679 upper=1.57079632679 effort=200 velocity=15 -> lower=-1.57079632679 upper=1.57079632679 effort=200 velocity=10
- joint SE: limit lower=-1.57079632679 upper=0.523598775598 effort=200 velocity=15 -> lower=-1.57079632679 upper=0.523598775598 effort=200 velocity=10
- joint WP: limit lower=-1.1 upper=0.581 effort=200 velocity=15 -> lower=-1.1 upper=0.581 effort=200 velocity=10
- joint WY: limit lower=-1.01 upper=0.675 effort=200 velocity=15 -> lower=-1.01 upper=0.675 effort=200 velocity=10
- joint linkage_bl: limit effort=200 velocity=15 -> effort=200 velocity=10
- joint linkage_tl: limit effort=200 velocity=15 -> effort=200 velocity=10
- joint linkage_tr: limit lower=-1.28 upper=1.0471975512 effort=200 velocity=15 -> lower=-1.28 upper=1.0471975512 effort=200 velocity=10

File: grips_description/urdf/common.xacro (robot description, xacro)
@@ -8,5 +8,5 @@
 	<property name="pi" value="3.1415926535897931" />
 	<property name="max_effort" value="200" />
-  <property name="max_velocity" value="15" />
+  <property name="max_velocity" value="10" />
 	<!-- Links Mass -->
 	<property name="base_mass" value="1.208" />

Commit message: Added bash script to generate the openrave kinematic reachability

File: grips_description/robots/bimanual.urdf (robot description, URDF)
Before this commit: robot bimanual, 35 links, 34 joints
Joints:
- joint left_WP: limit lower=-1.1 upper=0.581 effort=200 velocity=10 -> lower=-0.581 upper=1.1 effort=200 velocity=10
- joint right_WP: limit lower=-1.1 upper=0.581 effort=200 velocity=10 -> lower=-0.581 upper=1.1 effort=200 velocity=10

File: grips_description/robots/grips.urdf (robot description, URDF)
Before this commit: robot grips, 18 links, 17 joints
Joints:
- joint WP: limit lower=-1.1 upper=0.581 effort=200 velocity=10 -> lower=-0.581 upper=1.1 effort=200 velocity=10

File: grips_description/urdf/grips_macro.xacro (robot description, xacro)
@@ -77,5 +77,5 @@
       <axis xyz="1 0 0" />
       <origin xyz="0 0.26109 7.5e-3" rpy="0 0 0" />
-      <limit lower="-1.1" upper="0.581" effort="${max_effort}" velocity="${max_velocity}" />
+      <limit lower="-0.581" upper="1.1" effort="${max_effort}" velocity="${max_velocity}" />
       <dynamics damping="${WP_damping}"/>
     </joint>
