Commit message: Added ik_validation Added namespaces to better organization of the topics

File: grips_description/urdf/grips_macro.xacro (robot description, xacro)
@@ -53,5 +53,5 @@
       <axis xyz="0 0 1" />
       <origin xyz="0 0 15.24e-3" rpy="0 0 0" />
-      <limit lower="${-pi/2}" upper="${pi/2}" effort="${max_effort}" velocity="${max_velocity}" />
+      <limit lower="${-pi/2}" upper="${pi/2}" effort="${max_effort}" velocity="${80*pi/180}" />
       <dynamics damping="${SA_damping}"/>
     </joint>
@@ -61,5 +61,5 @@
       <axis xyz="1 0 0" />
       <origin xyz="0 0 0.33812" rpy="0 0 0" />
-      <limit lower="${-pi/2}" upper="${pi/6}" effort="${max_effort}" velocity="${max_velocity}" />
+      <limit lower="${-pi/2}" upper="${pi/6}" effort="${max_effort}" velocity="${65*pi/180}" />
       <dynamics damping="${SE_damping}" friction="10"/>
     </joint>
@@ -69,5 +69,5 @@
       <axis xyz="1 0 0" />
       <origin xyz="0 -9.82e-3 0.52167" rpy="0 0 0" />
-      <limit lower="-1.28" upper="${pi/3}" effort="${max_effort}" velocity="${max_velocity}" />
+      <limit lower="-1.28" upper="${pi/3}" effort="${max_effort}" velocity="${50*pi/180}" />
       <dynamics damping="10"/>
     </joint>
@@ -77,5 +77,5 @@
       <axis xyz="1 0 0" />
       <origin xyz="0 0.26109 7.5e-3" rpy="0 0 0" />
-      <limit lower="-0.581" upper="1.1" effort="${max_effort}" velocity="${max_velocity}" />
+      <limit lower="-0.581" upper="1.1" effort="${max_effort}" velocity="${100*pi/180}" />
       <dynamics damping="${WP_damping}"/>
     </joint>
@@ -85,5 +85,5 @@
       <axis xyz="0 0 1" />
       <origin xyz="0 0.13322 0" rpy="0 0 0" />
-      <limit lower="-1.01" upper="0.675" effort="${max_effort}" velocity="${max_velocity}" />
+      <limit lower="-1.01" upper="0.675" effort="${max_effort}" velocity="${115*pi/180}" />
       <dynamics damping="${WY_damping}"/>
     </joint>
@@ -93,5 +93,5 @@
       <axis xyz="0 1 0" />
       <origin xyz="-0.787e-3 0.190892 0.051331" rpy="0 0 0" />
-      <limit effort="${max_effort}" velocity="200" />
+      <limit effort="${max_effort}" velocity="${200*pi/180}" />
       <dynamics damping="${WR_damping}"/>
     </joint>
@@ -138,5 +138,5 @@
     <gazebo reference="${name}upper_arm">
       <material>Telerobcar/MetalSeamed</material>
-      <selfCollide>true</selfCollide>
+      <selfCollide>false</selfCollide>
     </gazebo>
     <gazebo reference="${name}elbow_pivot">
@@ -150,21 +150,21 @@
     <gazebo reference="${name}forearm">
       <material>Telerobcar/MetalSeamed</material>
-      <selfCollide>true</selfCollide>
+      <selfCollide>false</selfCollide>
     </gazebo>
     <gazebo reference="${name}pitch">
       <material>Telerobcar/MetalSeamed</material>
-      <selfCollide>true</selfCollide>
+      <selfCollide>false</selfCollide>
     </gazebo>
     <gazebo reference="${name}yaw">
       <material>Telerobcar/MetalSeamed</material>
-      <selfCollide>true</selfCollide>
+      <selfCollide>false</selfCollide>
     </gazebo>
     <gazebo reference="${name}end_effector">
-      <selfCollide>true</selfCollide>
+      <selfCollide>false</selfCollide>
     </gazebo>
     <!-- camera -->
     <gazebo reference="${name}camera">
       <material>Gazebo/FlatBlack</material>
-      <selfCollide>true</selfCollide>
+      <selfCollide>false</selfCollide>
       <sensor type="camera" name="${name}camera">
         <update_rate>30.0</update_rate>

File: grips_description/urdf/simple_gripper_macro.xacro (robot description, xacro)
@@ -86,5 +86,5 @@
     <gazebo reference="${name}gripper_base">
       <material>Telerobcar/MetalSeamed</material>
-      <selfCollide>true</selfCollide>
+      <selfCollide>false</selfCollide>
     </gazebo>
     <gazebo reference="${name}r_outer">

Commit message: [grips_kinematics] Fixed kinematic_services to make it general

File: grips_description/robots/bimanual.urdf (robot description, URDF)
Before this commit: robot bimanual, 35 links, 34 joints
Links:
- link left_base_link: geometry collision mesh filename=package://grips_description/meshes/collision/base.dae; visual mesh filename=package://grips_description/meshes/visual/base.dae
- link left_camera: geometry collision mesh filename=package://grips_description/meshes/collision/camera.dae; visual mesh filename=package://grips_description/meshes/visual/camera.dae
- link left_coupling: geometry collision mesh filename=package://grips_description/meshes/visual/coupling.dae; visual mesh filename=package://grips_description/meshes/visual/coupling.dae
- link left_elbow_pivot: geometry collision mesh filename=package://grips_description/meshes/visual/elbow_pivot.dae; visual mesh filename=package://grips_description/meshes/visual/elbow_pivot.dae
- link left_forearm: geometry collision mesh filename=package://grips_description/meshes/collision/forearm.dae; visual mesh filename=package://grips_description/meshes/visual/forearm.dae
- link left_gripper_base: geometry collision mesh filename=package://grips_description/meshes/visual/gripper_base.dae; visual mesh filename=package://grips_description/meshes/visual/gripper_base.dae
- link left_l_finger: geometry collision mesh filename=package://grips_description/meshes/visual/l_finger.dae; visual mesh filename=package://grips_description/meshes/visual/l_finger.dae
- link left_l_inner: geometry collision mesh filename=package://grips_description/meshes/visual/l_inner_pivot.dae; visual mesh filename=package://grips_description/meshes/visual/l_inner_pivot.dae
- link left_l_outer: geometry collision mesh filename=package://grips_description/meshes/visual/outer_pivot.dae; visual mesh filename=package://grips_description/meshes/visual/outer_pivot.dae
- link left_manifold: geometry collision mesh filename=package://grips_description/meshes/collision/manifold.dae; visual mesh filename=package://grips_description/meshes/visual/manifold.dae
- link left_pitch: geometry collision mesh filename=package://grips_description/meshes/collision/pitch.dae; visual mesh filename=package://grips_description/meshes/visual/pitch.dae
- link left_r_finger: geometry collision mesh filename=package://grips_description/meshes/visual/r_finger.dae; visual mesh filename=package://grips_description/meshes/visual/r_finger.dae
- link left_r_inner: geometry collision mesh filename=package://grips_description/meshes/visual/r_inner_pivot.dae; visual mesh filename=package://grips_description/meshes/visual/r_inner_pivot.dae
- link left_r_outer: geometry collision mesh filename=package://grips_description/meshes/visual/outer_pivot.dae; visual mesh filename=package://grips_description/meshes/visual/outer_pivot.dae
- link left_upper_arm: geometry collision mesh filename=package://grips_description/meshes/collision/upper_arm.dae; visual mesh filename=package://grips_description/meshes/visual/upper_arm.dae
- link left_yaw: geometry collision mesh filename=package://grips_description/meshes/collision/yaw.dae; visual mesh filename=package://grips_description/meshes/visual/yaw.dae
- link right_base_link: geometry collision mesh filename=package://grips_description/meshes/collision/base.dae; visual mesh filename=package://grips_description/meshes/visual/base.dae
- link right_camera: geometry collision mesh filename=package://grips_description/meshes/collision/camera.dae; visual mesh filename=package://grips_description/meshes/visual/camera.dae
- link right_coupling: geometry collision mesh filename=package://grips_description/meshes/visual/coupling.dae; visual mesh filename=package://grips_description/meshes/visual/coupling.dae
- link right_elbow_pivot: geometry collision mesh filename=package://grips_description/meshes/visual/elbow_pivot.dae; visual mesh filename=package://grips_description/meshes/visual/elbow_pivot.dae
- link right_forearm: geometry collision mesh filename=package://grips_description/meshes/collision/forearm.dae; visual mesh filename=package://grips_description/meshes/visual/forearm.dae
- link right_gripper_base: geometry collision mesh filename=package://grips_description/meshes/visual/gripper_base.dae; visual mesh filename=package://grips_description/meshes/visual/gripper_base.dae
- link right_l_finger: geometry collision mesh filename=package://grips_description/meshes/visual/l_finger.dae; visual mesh filename=package://grips_description/meshes/visual/l_finger.dae
- link right_l_inner: geometry collision mesh filename=package://grips_description/meshes/visual/l_inner_pivot.dae; visual mesh filename=package://grips_description/meshes/visual/l_inner_pivot.dae
- link right_l_outer: geometry collision mesh filename=package://grips_description/meshes/visual/outer_pivot.dae; visual mesh filename=package://grips_description/meshes/visual/outer_pivot.dae
- link right_manifold: geometry collision mesh filename=package://grips_description/meshes/collision/manifold.dae; visual mesh filename=package://grips_description/meshes/visual/manifold.dae
- link right_pitch: geometry collision mesh filename=package://grips_description/meshes/collision/pitch.dae; visual mesh filename=package://grips_description/meshes/visual/pitch.dae
- link right_r_finger: geometry collision mesh filename=package://grips_description/meshes/visual/r_finger.dae; visual mesh filename=package://grips_description/meshes/visual/r_finger.dae
- link right_r_inner: geometry collision mesh filename=package://grips_description/meshes/visual/r_inner_pivot.dae; visual mesh filename=package://grips_description/meshes/visual/r_inner_pivot.dae
- link right_r_outer: geometry collision mesh filename=package://grips_description/meshes/visual/outer_pivot.dae; visual mesh filename=package://grips_description/meshes/visual/outer_pivot.dae
- link right_upper_arm: geometry collision mesh filename=package://grips_description/meshes/collision/upper_arm.dae; visual mesh filename=package://grips_description/meshes/visual/upper_arm.dae
- link right_yaw: geometry collision mesh filename=package://grips_description/meshes/collision/yaw.dae; visual mesh filename=package://grips_description/meshes/visual/yaw.dae

File: grips_description/robots/grips.urdf (robot description, URDF)
Before this commit: robot grips, 18 links, 17 joints
Links:
- link base_link: geometry collision mesh filename=package://grips_description/meshes/collision/base.dae; visual mesh filename=package://grips_description/meshes/visual/base.dae
- link camera: geometry collision mesh filename=package://grips_description/meshes/collision/camera.dae; visual mesh filename=package://grips_description/meshes/visual/camera.dae
- link coupling: geometry collision mesh filename=package://grips_description/meshes/visual/coupling.dae; visual mesh filename=package://grips_description/meshes/visual/coupling.dae
- link elbow_pivot: geometry collision mesh filename=package://grips_description/meshes/visual/elbow_pivot.dae; visual mesh filename=package://grips_description/meshes/visual/elbow_pivot.dae
- link forearm: geometry collision mesh filename=package://grips_description/meshes/collision/forearm.dae; visual mesh filename=package://grips_description/meshes/visual/forearm.dae
- link gripper_base: geometry collision mesh filename=package://grips_description/meshes/visual/gripper_base.dae; visual mesh filename=package://grips_description/meshes/visual/gripper_base.dae
- link l_finger: geometry collision mesh filename=package://grips_description/meshes/visual/l_finger.dae; visual mesh filename=package://grips_description/meshes/visual/l_finger.dae
- link l_inner: geometry collision mesh filename=package://grips_description/meshes/visual/l_inner_pivot.dae; visual mesh filename=package://grips_description/meshes/visual/l_inner_pivot.dae
- link l_outer: geometry collision mesh filename=package://grips_description/meshes/visual/outer_pivot.dae; visual mesh filename=package://grips_description/meshes/visual/outer_pivot.dae
- link manifold: geometry collision mesh filename=package://grips_description/meshes/collision/manifold.dae; visual mesh filename=package://grips_description/meshes/visual/manifold.dae
- link pitch: geometry collision mesh filename=package://grips_description/meshes/collision/pitch.dae; visual mesh filename=package://grips_description/meshes/visual/pitch.dae
- link r_finger: geometry collision mesh filename=package://grips_description/meshes/visual/r_finger.dae; visual mesh filename=package://grips_description/meshes/visual/r_finger.dae
- link r_inner: geometry collision mesh filename=package://grips_description/meshes/visual/r_inner_pivot.dae; visual mesh filename=package://grips_description/meshes/visual/r_inner_pivot.dae
- link r_outer: geometry collision mesh filename=package://grips_description/meshes/visual/outer_pivot.dae; visual mesh filename=package://grips_description/meshes/visual/outer_pivot.dae
- link upper_arm: geometry collision mesh filename=package://grips_description/meshes/collision/upper_arm.dae; visual mesh filename=package://grips_description/meshes/visual/upper_arm.dae
- link yaw: geometry collision mesh filename=package://grips_description/meshes/collision/yaw.dae; visual mesh filename=package://grips_description/meshes/visual/yaw.dae

File: grips_description/robots/grips_robotiq.urdf (robot description, URDF)
Before this commit: robot grips, 13 links, 12 joints
Links:
- added link finger_1_link_0, mass 0.05; collision mesh filename=package://robotiq_s_model_visualization/meshes/s-model_arti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; visual mesh filename=package://robotiq_s_model_visualization/meshes/s-model_arti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
- added link finger_1_link_1, mass 0.15; collision mesh filename=package://robotiq_s_model_visualization/meshes/s-model_arti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; visual mesh filename=package://robotiq_s_model_visualization/meshes/s-model_arti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
- added link finger_1_link_2, mass 0.15; collision mesh filename=package://robotiq_s_model_visualization/meshes/s-model_arti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; visual mesh filename=package://robotiq_s_model_visualization/meshes/s-model_arti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
- added link finger_1_link_3, mass 0.05; collision mesh filename=package://robotiq_s_model_visualization/meshes/s-model_arti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; visual mesh filename=package://robotiq_s_model_visualization/meshes/s-model_arti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
- added link finger_2_link_0, mass 0.05; collision mesh filename=package://robotiq_s_model_visualization/meshes/s-model_arti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; visual mesh filename=package://robotiq_s_model_visualization/meshes/s-model_arti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
- added link finger_2_link_1, mass 0.15; collision mesh filename=package://robotiq_s_model_visualization/meshes/s-model_arti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; visual mesh filename=package://robotiq_s_model_visualization/meshes/s-model_arti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
- added link finger_2_link_2, mass 0.15; collision mesh filename=package://robotiq_s_model_visualization/meshes/s-model_arti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; visual mesh filename=package://robotiq_s_model_visualization/meshes/s-model_arti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
- added link finger_2_link_3, mass 0.05; collision mesh filename=package://robotiq_s_model_visualization/meshes/s-model_arti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; visual mesh filename=package://robotiq_s_model_visualization/meshes/s-model_arti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
- added link finger_middle_link_0, mass 0.05; collision mesh filename=package://robotiq_s_model_visualization/meshes/s-model_arti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; visual mesh filename=package://robotiq_s_model_visualization/meshes/s-model_arti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
- added link finger_middle_link_1, mass 0.15; collision mesh filename=package://robotiq_s_model_visualization/meshes/s-model_arti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; visual mesh filename=package://robotiq_s_model_visualization/meshes/s-model_arti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
- added link finger_middle_link_2, mass 0.15; collision mesh filename=package://robotiq_s_model_visualization/meshes/s-model_arti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; visual mesh filename=package://robotiq_s_model_visualization/meshes/s-model_arti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
- added link finger_middle_link_3, mass 0.05; collision mesh filename=package://robotiq_s_model_visualization/meshes/s-model_arti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; visual mesh filename=package://robotiq_s_model_visualization/meshes/s-model_arti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
- added link ft_end_effector
- added link ft_robotiq_plate, mass 0.2304; collision mesh filename=package://grips_description/meshes/visual/ft_robotiq_plate.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; visual mesh filename=package://grips_description/meshes/visual/ft_robotiq_plate.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
- added link ft_sensor, mass 0.2396; collision mesh filename=package://grips_description/meshes/visual/ft_sensor.dae; visual mesh filename=package://grips_description/meshes/visual/ft_sensor.dae
- added link palm; collision mesh filename=package://robotiq_s_model_visualization/meshes/s-model_arti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; visual mesh filename=package://robotiq_s_model_visualization/meshes/s-model_arti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
Joints:
- added joint finger_1_joint_1: type revolute, parent finger_1_link_0, child finger_1_link_1, origin xyz=0.020 0 0 rpy=0 0 0, axis 0 0 1, limit lower=0 upper=3.1416 effort=100 velocity=100
- added joint finger_1_joint_2: type revolute, parent finger_1_link_1, child finger_1_link_2, origin xyz=0.050 -.028 0 rpy=0 0 -0.52, axis 0 0 1, limit lower=0 upper=3.1416 effort=100 velocity=100
- added joint finger_1_joint_3: type revolute, parent finger_1_link_2, child finger_1_link_3, origin xyz=0.039 0 0 rpy=0 0 0, axis 0 0 1, limit lower=0 upper=3.1416 effort=100 velocity=100
- added joint finger_2_joint_1: type revolute, parent finger_2_link_0, child finger_2_link_1, origin xyz=0.020 0 0 rpy=0 0 0, axis 0 0 1, limit lower=0 upper=3.1416 effort=100 velocity=100
- added joint finger_2_joint_2: type revolute, parent finger_2_link_1, child finger_2_link_2, origin xyz=0.050 -.028 0 rpy=0 0 -0.52, axis 0 0 1, limit lower=0 upper=3.1416 effort=100 velocity=100
- added joint finger_2_joint_3: type revolute, parent finger_2_link_2, child finger_2_link_3, origin xyz=0.039 0 0 rpy=0 0 0, axis 0 0 1, limit lower=0 upper=3.1416 effort=100 velocity=100
- added joint finger_middle_joint_1: type revolute, parent finger_middle_link_0, child finger_middle_link_1, origin xyz=0.020 0 0 rpy=0 0 0, axis 0 0 1, limit lower=0 upper=3.1416 effort=100 velocity=100
- added joint finger_middle_joint_2: type revolute, parent finger_middle_link_1, child finger_middle_link_2, origin xyz=0.050 -.028 0 rpy=0 0 -0.52, axis 0 0 1, limit lower=0 upper=3.1416 effort=100 velocity=100
- added joint finger_middle_joint_3: type revolute, parent finger_middle_link_2, child finger_middle_link_3, origin xyz=0.039 0 0 rpy=0 0 0, axis 0 0 1, limit lower=0 upper=3.1416 effort=100 velocity=100
- added joint ft_end_joint: type fixed, parent ft_robotiq_plate, child ft_end_effector, origin xyz=0 0 0 rpy=-1.57079632679 0 0
- added joint ft_plate_joint: type fixed, parent ft_sensor, child ft_robotiq_plate, origin xyz=0 -11e-3 0 rpy=-1.57079632679 0 0
- added joint ft_sensor_joint: type fixed, parent ft_wrist_plate, child ft_sensor, origin xyz=0 0 0.0564 rpy=-1.57079632679 0 0
- added joint palm_finger_1_joint: type revolute, parent palm, child finger_1_link_0, origin xyz=-0.0455 0.0214 0.036 rpy=0 3.1416 -1.57, axis 0 1 0, limit lower=-0.16 upper=0.25 effort=100 velocity=100
- added joint palm_finger_2_joint: type revolute, parent palm, child finger_2_link_0, origin xyz=-0.0455 0.0214 -0.036 rpy=0 3.1416 -1.57, axis 0 1 0, limit lower=-0.25 upper=0.16 effort=100 velocity=100
- added joint palm_finger_middle_joint: type fixed, parent palm, child finger_middle_link_0, origin xyz=0.0455 0.0214 0 rpy=0 0 1.57, axis 0 0 1
- added joint robotiq_anchor: type fixed, parent ft_end_effector, child palm, origin xyz=0 54e-3 0 rpy=0 0 0
- joint ft_wrist_joint: origin xyz=0 4.7e-3 0 rpy=$0 0 0 -> xyz=0 0 0 rpy=0 0 0
