Commit message: Added bimanual visualization

File: grips_description/robots/bimanual.urdf (robot description, URDF)
Before this commit: robot bimanual, 35 links, 34 joints
Links:
- removed link left_coupling
- removed link left_elbow_pivot
- removed link right_coupling
- removed link right_elbow_pivot
Joints:
- removed joint left_linkage_bl
- removed joint left_linkage_tl
- removed joint right_linkage_bl
- removed joint right_linkage_tl

File: grips_description/robots/bimanual.xacro (robot description, xacro)
@@ -1,12 +1,12 @@
 <?xml version="1.0"?>
 <robot name="bimanual" xmlns:xacro="http://www.ros.org/wiki/xacro">
-	<!-- Import common macros-->
-	<xacro:include filename="$(find grips_description)/urdf/common.xacro" />
-	<!-- Import materials for rviz-->
-	<xacro:include filename="$(find grips_description)/urdf/materials.xacro" />
-	<!-- Import robot without gripper -->
-	<xacro:include filename="$(find grips_description)/urdf/grips_macro.xacro" />
-	<!-- Import simple gripper -->
-	<xacro:include filename="$(find grips_description)/urdf/simple_gripper_macro.xacro" />
+  <!-- Import common macros-->
+  <xacro:include filename="$(find grips_description)/urdf/common.xacro" />
+  <!-- Import materials for rviz-->
+  <xacro:include filename="$(find grips_description)/urdf/materials.xacro" />
+  <!-- Import robot without gripper -->
+  <xacro:include filename="$(find grips_description)/urdf/grips_macro.xacro" />
+  <!-- Import simple gripper -->
+  <xacro:include filename="$(find grips_description)/urdf/simple_gripper_macro.xacro" />
   <!-- Create the grips robots -->
   <grips_robot name="left_"/>
@@ -16,30 +16,30 @@
   <simple_gripper name="right_"/>
   <!-- Fix the grippers to the robot -->
-	<joint name="left_gripper_anchor" type="fixed">
-		<origin xyz="0 0 0" rpy="0 0 0" />
-		<parent link="left_end_effector" />
-		<child link="left_gripper_base" />
-	</joint>
-	<joint name="right_gripper_anchor" type="fixed">
-		<origin xyz="0 0 0" rpy="0 0 0" />
-		<parent link="right_end_effector" />
-		<child link="right_gripper_base" />
-	</joint>
-	<!-- Used for fixing the robots to Gazebo -->
-	<link name="world" />
-	<joint name="left_anchor" type="fixed">
-		<origin xyz="0 0 0.801" rpy="0 0 0" />
-		<parent link="world" />
-		<child link="left_base_link" />
-	</joint>
-	<joint name="right_anchor" type="fixed">
-		<origin xyz="1 0 0.801" rpy="0 0 0" />
-		<parent link="world" />
-		<child link="right_base_link" />
-	</joint>
-	<!-- ros_control plugin -->
-	<gazebo>
-		<plugin name="ros_control" filename="libgazebo_ros_control.so">
-		</plugin>
-	</gazebo>
+  <joint name="left_gripper_anchor" type="fixed">
+    <origin xyz="0 0 0" rpy="0 0 0" />
+    <parent link="left_end_effector" />
+    <child link="left_gripper_base" />
+  </joint>
+  <joint name="right_gripper_anchor" type="fixed">
+    <origin xyz="0 0 0" rpy="0 0 0" />
+    <parent link="right_end_effector" />
+    <child link="right_gripper_base" />
+  </joint>
+  <!-- Used for fixing the robots to Gazebo -->
+  <link name="world" />
+  <joint name="left_anchor" type="fixed">
+    <origin xyz="0 0 0.801" rpy="0 0 0" />
+    <parent link="world" />
+    <child link="left_base_link" />
+  </joint>
+  <joint name="right_anchor" type="fixed">
+    <origin xyz="1 0 0.801" rpy="0 0 0" />
+    <parent link="world" />
+    <child link="right_base_link" />
+  </joint>
+  <!-- ros_control plugin -->
+  <gazebo>
+    <plugin name="ros_control" filename="libgazebo_ros_control.so">
+    </plugin>
+  </gazebo>
 </robot>

File: grips_description/robots/grips_robotiq.urdf (robot description, URDF)
Before this commit: robot grips, 29 links, 28 joints
Links:
- removed link coupling
- removed link elbow_pivot
Joints:
- removed joint linkage_bl
- removed joint linkage_tl

File: grips_description/urdf/grips_macro.xacro (robot description, xacro)
@@ -17,12 +17,4 @@
       <upper_arm_inertia />
     </link_collision>
-    <!-- elbow pivot link -->
-    <create_link name="${name}elbow_pivot" color="black" mesh="${elbow_pivot_mesh}" cog="${elbow_pivot_cog}" mass="${elbow_pivot_mass}" >
-      <elbow_pivot_inertia />
-    </create_link>
-    <!-- coupling link -->
-    <create_link name="${name}coupling" color="black" mesh="${coupling_mesh}" cog="${coupling_cog}" mass="${coupling_mass}" >
-      <coupling_inertia />
-    </create_link>
     <!-- forearm link -->
     <link_collision name="${name}forearm" color="black" mesh="${forearm_mesh}" cog="${forearm_cog}" mass="${forearm_mass}" >
@@ -42,9 +34,4 @@
     <!-- end effector dummy link -->
     <link name="${name}end_effector" />
-    <!-- camera link -->
-    <link_collision name="${name}camera" color="black" mesh="${camera_mesh}" cog="${camera_cog}" mass="${camera_mass}" >
-      <mesh filename="package://grips_description/meshes/collision/camera.dae" />
-      <camera_inertia />
-    </link_collision>
     <!-- Joints -->
     <joint name="${name}SA" type="revolute">
@@ -96,27 +83,4 @@
       <dynamics damping="${WR_damping}"/>
     </joint>
-    <joint name="${name}camera_joint" type="fixed">
-      <child link="${name}camera"/>
-      <parent link="${name}yaw"/>
-      <axis xyz="0 1 0" />
-      <origin xyz="0 ${0.190892/2} 0.25" rpy="0 ${pi/6} ${pi/2}"/>
-    </joint>
-    <!-- four-bar linkage -->
-    <joint name="${name}linkage_tl" type="continuous">
-      <child link="${name}coupling" />
-      <parent link="${name}forearm" />
-      <axis xyz="1 0 0" />
-      <origin xyz="0 -0.123444 0.029845" rpy="0.019320795 0 0" />
-      <limit effort="${max_effort}" velocity="${max_velocity}" />
-      <dynamics damping="${linkage_damping}" friction="${linkage_friction}"/>
-    </joint>
-    <joint name="${name}linkage_bl" type="continuous">
-      <child link="${name}elbow_pivot" />
-      <parent link="${name}coupling" />
-      <axis xyz="1 0 0" />
-      <origin xyz="0 0 -0.5207" rpy="-0.24521876 0 0" />
-      <limit effort="${max_effort}" velocity="${max_velocity}" />
-      <dynamics damping="${linkage_damping}" friction="${linkage_friction}"/>
-    </joint>
     <!-- Transmissions -->
     <simple_transmission joint="${name}SA" />
@@ -126,6 +90,4 @@
     <simple_transmission joint="${name}WR" />
     <simple_transmission joint="${name}linkage_tr" />
-    <simple_transmission joint="${name}linkage_tl" />
-    <simple_transmission joint="${name}linkage_bl" />
     <gazebo reference="${name}base_link">
       <material>Telerobcar/MetalSeamed</material>
@@ -137,12 +99,4 @@
     </gazebo>
     <gazebo reference="${name}upper_arm">
-      <material>Telerobcar/MetalSeamed</material>
-      <selfCollide>false</selfCollide>
-    </gazebo>
-    <gazebo reference="${name}elbow_pivot">
-      <material>Telerobcar/MetalSeamed</material>
-      <selfCollide>false</selfCollide>
-    </gazebo>
-    <gazebo reference="${name}coupling">
       <material>Telerobcar/MetalSeamed</material>
       <selfCollide>false</selfCollide>
@@ -163,38 +117,4 @@
       <selfCollide>false</selfCollide>
     </gazebo>
-    <!-- camera -->
-    <gazebo reference="${name}camera">
-      <material>Gazebo/FlatBlack</material>
-      <selfCollide>false</selfCollide>
-      <sensor type="camera" name="${name}camera">
-        <update_rate>30.0</update_rate>
-        <camera name="${name}camera">
-          <horizontal_fov>1.3962634</horizontal_fov>
-          <image>
-            <width>800</width>
-            <height>800</height>
-            <format>R8G8B8</format>
-          </image>
-          <clip>
-            <near>0.02</near>
-            <far>300</far>
-          </clip>
-        </camera>
-        <plugin name="camera_controller" filename="libgazebo_ros_camera.so">
-          <alwaysOn>true</alwaysOn>
-          <updateRate>0.0</updateRate>
-          <cameraName>${name}camera</cameraName>
-          <imageTopicName>image_raw</imageTopicName>
-          <cameraInfoTopicName>camera_info</cameraInfoTopicName>
-          <frameName>${name}camera</frameName>
-          <hackBaseline>0.07</hackBaseline>
-          <distortionK1>0.0</distortionK1>
-          <distortionK2>0.0</distortionK2>
-          <distortionK3>0.0</distortionK3>
-          <distortionT1>0.0</distortionT1>
-          <distortionT2>0.0</distortionT2>
-        </plugin>
-      </sensor>
-    </gazebo>
   </macro>
 </robot>
