Commit message: Changed gazebo inertia values and cleaned-up the repo

File: grips_description/robots/grips_no_gripper.urdf.xacro (robot description, xacro)
@@ -12,3 +12,7 @@
   <link name="world" />
   <serial_arm parent="world"/>
+  <!-- ros_control plugin  -->
+  <gazebo>
+    <plugin name="ros_control" filename="libgazebo_ros_control.so"/>
+  </gazebo>
 </robot>

File: grips_description/urdf/common.xacro (robot description, xacro)
@@ -8,15 +8,23 @@
   <property name="max_velocity" value="5" />
   <!-- Macros -->
-  <!-- Inertia Macro -->
-  <macro name="cylinder_inertial" params="cog mass radius length">
+  <macro name="cylinder_collision" params="radius length">
+    <collision>
+      <origin xyz="0 0 ${length/2}" rpy="0 0 0"/>
+      <geometry>
+        <cylinder radius="${radius}" length="${length}"/>
+      </geometry>
+    </collision>
+  </macro>
+  <macro name="cylinder_inertia" params="mass radius length">
     <inertial>
-      <origin xyz="${cog}" rpy="0 0 0" />
+      <origin xyz="0 0 ${length/2}" rpy="0 0 0" />
       <mass value="${mass}" />
-      <inertia  ixx="${3*mass*radius^2 / 12  + length^2 / 12}" ixy="0.0"  ixz="0.0"
-                iyy="${3*mass*radius^2 / 12  + length^2 / 12}" iyz="0.0"  izz="${mass*radius^2 / 2}" />
+      <inertia  ixx="${mass*radius^2 / 4  + mass*length^2 / 12}" ixy="0.0"  ixz="0.0"
+                iyy="${mass*radius^2 / 4  + mass*length^2 / 12}" iyz="0.0"
+                izz="${mass*radius^2 / 2}" />
     </inertial>
   </macro>
   <!-- Link Macro -->
-  <macro name="create_link" params="name color mesh *inertia">
+  <macro name="create_link" params="name color mesh *collision *inertia">
     <link name="${name}">
       <visual>
@@ -26,12 +34,23 @@
         <material name="${color}" />
       </visual>
-<!--
+      <xacro:insert_block name="collision" />
+      <xacro:insert_block name="inertia" />
+    </link>
+  </macro>
+  <!-- A smaller dummy link makes the model to explode in Gazebo -->
+  <macro name="dummy_link" params="name">
+    <link name="${name}">
+      <visual>
+        <geometry>
+          <sphere radius="0.02"/>
+        </geometry>
+        <material name="black" />
+      </visual>
       <collision>
         <geometry>
-          <mesh filename="${mesh}" />
+          <sphere radius="0.02"/>
         </geometry>
       </collision>
-      <xacro:insert_block name="inertia" />
--->
+      <cylinder_inertia radius="0.02" length="0.02" mass="0.05"/>
     </link>
   </macro>

File: grips_description/urdf/serial_arm.xacro (robot description, xacro)
@@ -2,8 +2,16 @@
 <robot xmlns:xacro="http://www.ros.org/wiki/xacro">
   <!-- Dimensions -->
-  <property name="base_radius" value="0.085" />
+  <property name="base_radius" value="0.125" />
   <property name="base_length" value="15.24e-3" />
-  <property name="manifold_radius" value="0.2" />
+  <property name="manifold_radius" value="0.205" />
   <property name="manifold_length" value="0.33812" />
+  <property name="upper_arm_radius" value="0.075" />
+  <property name="upper_arm_length" value="0.52167" />
+  <property name="forearm_radius" value="0.075" />
+  <property name="forearm_length" value="0.385078" />
+  <property name="pitch_radius" value="0.075" />
+  <property name="pitch_length" value="0.133223" />
+  <property name="yaw_radius" value="0.085" />
+  <property name="yaw_length" value="0.190892" />
   <!-- Link Masses -->
   <property name="base_mass" value="1.208" />
@@ -16,14 +24,4 @@
   <property name="yaw_mass" value="4.689" />
   <property name="camera_mass" value="0.869" />
-  <!-- Link COGs -->
-  <property name="base_cog" value="0 0 7e-3" />
-  <property name="manifold_cog" value="0 2e-3 0.21" />
-  <property name="upper_arm_cog" value="0 5e-3 0.227" />
-  <property name="elbow_pivot_cog" value="-3.6e-10 80.686e-3 -6.33e-5" />
-  <property name="coupling_cog" value="0 0 -0.26035" />
-  <property name="forearm_cog" value="0 0.155337 0.012119" />
-  <property name="pitch_cog" value="0 0.065 0" />
-  <property name="yaw_cog" value="-1e-3 95.791e-3 18.273e-3" />
-  <property name="camera_cog" value="0.077 0.007 0.002" />
   <!-- Meshes -->
   <property name="base_mesh" value="package://grips_description/meshes/visual/base.dae" />
@@ -46,24 +44,62 @@
   <macro name="serial_arm" params="parent">
     <create_link name="base_link" color="black" mesh="${base_mesh}" >
-      <cylinder_inertial cog="${base_cog}" mass="${base_mass}" radius="${base_radius}" length="${base_length}"/>
+      <cylinder_collision radius="${base_radius}" length="${base_length}" />
+      <cylinder_inertia radius="${base_radius}" length="${base_length}" mass="${base_mass}"/>
     </create_link>
-    <create_link name="manifold" color="blue" mesh="${manifold_mesh}" >
-      <cylinder_inertial cog="${manifold_cog}" mass="${manifold_mass}" radius="${manifold_radius}" length="${manifold_length}"/>
+    <create_link name="manifold" color="black" mesh="${manifold_mesh}" >
+      <cylinder_collision radius="${manifold_radius}" length="${manifold_length}" />
+      <cylinder_inertia radius="${manifold_radius}" length="${manifold_length}" mass="${manifold_mass}"/>
     </create_link>
-<!--
-    <create_link name="upper_arm" color="black" mesh="${upper_arm_mesh}" cog="${upper_arm_cog}" mass="${upper_arm_mass}" >
-      <upper_arm_inertia />
+    <create_link name="upper_arm" color="black" mesh="${upper_arm_mesh}" >
+      <cylinder_collision radius="${upper_arm_radius}" length="${upper_arm_length}" />
+      <cylinder_inertia radius="${upper_arm_radius}" length="${upper_arm_length}" mass="${upper_arm_mass}"/>
     </create_link>
-    <create_link name="forearm" color="black" mesh="${forearm_mesh}" cog="${forearm_cog}" mass="${forearm_mass}" >
-      <forearm_inertia />
+    <create_link name="forearm" color="black" mesh="${forearm_mesh}" >
+      <collision>
+        <origin xyz="0 ${forearm_length/2 - 0.1234} 0" rpy="${pi/2} 0 0"/>
+        <geometry>
+          <cylinder radius="${forearm_radius}" length="${forearm_length}"/>
+        </geometry>
+      </collision>
+      <inertial>
+        <origin xyz="0 ${forearm_length/2 - 0.1234} 0" rpy="0 0 0"/>
+        <mass value="${forearm_mass}" />
+        <inertia  ixx="${forearm_mass*forearm_radius^2 / 4  + forearm_mass*forearm_length^2 / 12}" ixy="0.0"  ixz="0.0"
+                  iyy="${forearm_mass*forearm_radius^2 / 2}" iyz="0.0"
+                  izz="${forearm_mass*forearm_radius^2 / 4  + forearm_mass*forearm_length^2 / 12}" />
+      </inertial>
     </create_link>
-    <create_link name="pitch" color="black" mesh="${pitch_mesh}">
-      <pitch_inertia />
+    <create_link name="pitch" color="black" mesh="${pitch_mesh}" >
+      <collision>
+        <origin xyz="0 ${pitch_length/2} 0" rpy="${pi/2} 0 0"/>
+        <geometry>
+          <cylinder radius="${pitch_radius}" length="${pitch_length}"/>
+        </geometry>
+      </collision>
+      <inertial>
+        <origin xyz="0 ${pitch_length/2} 0" rpy="0 0 0"/>
+        <mass value="${pitch_mass}" />
+        <inertia  ixx="${pitch_mass*pitch_radius^2 / 4  + pitch_mass*pitch_length^2 / 12}" ixy="0.0"  ixz="0.0"
+                  iyy="${pitch_mass*pitch_radius^2 / 2}" iyz="0.0"
+                  izz="${pitch_mass*pitch_radius^2 / 4  + pitch_mass*pitch_length^2 / 12}" />
+      </inertial>
     </create_link>
-    <create_link name="yaw" color="black" mesh="${yaw_mesh}">
-      <yaw_inertia />
+    <create_link name="yaw" color="black" mesh="${yaw_mesh}" >
+      <collision>
+        <origin xyz="0 ${yaw_length/2} 0" rpy="${pi/2} 0 0"/>
+        <geometry>
+          <cylinder radius="${yaw_radius}" length="${yaw_length}"/>
+        </geometry>
+      </collision>
+      <inertial>
+        <origin xyz="0 ${yaw_length/2} 0" rpy="0 0 0"/>
+        <mass value="${yaw_mass}" />
+        <inertia  ixx="${yaw_mass*yaw_radius^2 / 4  + yaw_mass*yaw_length^2 / 12}" ixy="0.0"  ixz="0.0"
+                  iyy="${yaw_mass*yaw_radius^2 / 2}" iyz="0.0"
+                  izz="${yaw_mass*yaw_radius^2 / 4  + yaw_mass*yaw_length^2 / 12}" />
+      </inertial>
     </create_link>
-    <link name="end_effector" />
--->
+    <!-- This dummy link is needed for coupling hands to the robot -->
+    <dummy_link name="end_effector" />
     <!-- Joints -->
     <joint name="anchor" type="fixed">
@@ -80,10 +116,9 @@
       <dynamics damping="${SA_damping}"/>
     </joint>
-<!--
     <joint name="SE" type="revolute">
       <child link="upper_arm" />
       <parent link="manifold" />
       <axis xyz="1 0 0" />
-      <origin xyz="0 0 0.33812" rpy="0 0 0" />
+      <origin xyz="0 0 ${manifold_length}" rpy="0 0 0" />
       <limit lower="${-pi/2}" upper="${pi/6}" effort="${max_effort}" velocity="${65*pi/180}" />
       <dynamics damping="${SE_damping}" friction="10"/>
@@ -93,5 +128,5 @@
       <parent link="upper_arm" />
       <axis xyz="1 0 0" />
-      <origin xyz="0 -9.82e-3 0.52167" rpy="0 0 0" />
+      <origin xyz="0 -9.82e-3 ${upper_arm_length}" rpy="0 0 0" />
       <limit lower="-1.28" upper="${pi/3}" effort="${max_effort}" velocity="${50*pi/180}" />
       <dynamics damping="10"/>
@@ -109,5 +144,5 @@
       <parent link="pitch" />
       <axis xyz="0 0 1" />
-      <origin xyz="0 0.13322 0" rpy="0 0 0" />
+      <origin xyz="0 ${pitch_length} 0" rpy="0 0 0" />
       <limit lower="-1.01" upper="0.675" effort="${max_effort}" velocity="${115*pi/180}" />
       <dynamics damping="${WY_damping}"/>
@@ -117,16 +152,15 @@
       <parent link="yaw" />
       <axis xyz="0 1 0" />
-      <origin xyz="-0.787e-3 0.190892 0.051331" rpy="0 0 0" />
+      <origin xyz="-0.787e-3 ${yaw_length} 0.051331" rpy="0 0 0" />
       <limit effort="${max_effort}" velocity="${200*pi/180}" />
       <dynamics damping="${WR_damping}"/>
     </joint>
--->
-    <!-- Transmissions
+    <!-- Transmissions -->
     <simple_transmission joint="SA" />
     <simple_transmission joint="SE" />
+    <simple_transmission joint="linkage_tr" />
     <simple_transmission joint="WP" />
     <simple_transmission joint="WY" />
     <simple_transmission joint="WR" />
-    <simple_transmission joint="linkage_tr" /> -->
     <gazebo reference="base_link">
       <material>Telerobcar/MetalSeamed</material>
