Commit message: Added F/T sensor model to gazebo (not the plugin) for controlling the robot in the sensor reference frame

File: grips_description/robots/grips_robotiq.urdf.xacro (robot description, xacro)
@@ -6,34 +6,15 @@
   <xacro:include filename="$(find grips_description)/urdf/materials.xacro" />
   <!-- Import robot without gripper -->
-  <xacro:include filename="$(find grips_description)/urdf/grips_macro.xacro" />
+  <xacro:include filename="$(find grips_description)/urdf/serial_arm.xacro" />
   <!-- Import ft sensor -->
   <xacro:include filename="$(find grips_description)/urdf/ftsensor.xacro" />
-  <!-- Import robotiq s model -->
-  <xacro:include filename="$(find robotiq_s_model_visualization)/cfg/s-model_articulated_macro.xacro" />
-  <property name="robot_name" value="" />
   <!-- Create the grips robot -->
-  <grips_robot name="${robot_name}"/>
-  <!-- Used for fixing robot to Gazebo 'base_link' -->
   <link name="world" />
-  <joint name="anchor" type="fixed">
-    <origin xyz="0 0 0.001" rpy="0 0 0" />
-    <parent link="world" />
-    <child link="base_link" />
-  </joint>
+  <serial_arm parent="world"/>
   <!-- Add the ft_sensor -->
-  <ftsensor name="${robot_name}" parent="end_effector"/>
-   Add robotiq hand
-  <s-model_articulated prefix=""/>
-  <!-- Used for fixing Robotiq to the FT sensor -->
-  <joint name="robotiq_anchor" type="fixed">
-    <origin xyz="0 54e-3 0" rpy="0 0 0" />
-    <parent link="ft_end_effector" />
-    <child link="palm" />
-  </joint>
-  <!-- ros_control plugin -->
+  <ftsensor parent="end_effector"/>
+  <!-- ros_control plugin  -->
   <gazebo>
-    <plugin name="ros_control" filename="libgazebo_ros_control.so">
-      <robotNamespace>/grips_robotiq</robotNamespace>
-    </plugin>
+    <plugin name="ros_control" filename="libgazebo_ros_control.so"/>
   </gazebo>
 </robot>

File: grips_description/urdf/common.xacro (robot description, xacro)
@@ -43,14 +43,14 @@
       <visual>
         <geometry>
-          <sphere radius="0.02"/>
+          <sphere radius="0.01"/>
         </geometry>
-        <material name="black" />
+        <material name="blue" />
       </visual>
       <collision>
         <geometry>
-          <sphere radius="0.02"/>
+          <sphere radius="0.01"/>
         </geometry>
       </collision>
-      <cylinder_inertia radius="0.02" length="0.02" mass="0.05"/>
+      <cylinder_inertia radius="0.01" length="0.02" mass="0.05"/>
     </link>
   </macro>

File: grips_description/urdf/ftsensor.xacro (robot description, xacro)
@@ -2,77 +2,86 @@
 <robot xmlns:xacro="http://www.ros.org/wiki/xacro">
   <!-- Meshes -->
-  <property name="ft_kraft_plate_mesh"   value="package://grips_description/meshes/visual/ft_kraft_plate.dae" />
-  <property name="ft_robotiq_plate_mesh" value="package://grips_description/meshes/visual/ft_robotiq_plate.dae" />
+  <property name="wrist_coupling_mesh"   value="package://grips_description/meshes/visual/wrist_coupling.dae" />
+  <property name="ft_coupling_mesh"   value="package://grips_description/meshes/visual/ft_coupling.dae" />
   <property name="ft_sensor_mesh"        value="package://grips_description/meshes/visual/ft_sensor.dae" />
-  <property name="ft_wrist_plate_mesh"   value="package://grips_description/meshes/visual/ft_wrist_plate.dae" />
+  <property name="robotiq_coupling_mesh" value="package://grips_description/meshes/visual/robotiq_coupling.dae" />
+  <!-- Dimensions -->
+  <property name="wrist_coupling_radius" value="23.8e-3" />
+  <property name="wrist_coupling_length" value="19e-3" />
+  <property name="ft_coupling_radius" value="33.7e-3" />
+  <property name="ft_coupling_length" value="19e-3" />
+  <property name="ft_sensor_radius" value="37e-3" />
+  <property name="ft_sensor_length" value="28e-3" />
   <!-- Links Mass -->
-  <property name="ft_kraft_plate_mass"    value="0.059" />    <!-- Density: 5000 kg/m3 -->
-  <property name="ft_robotiq_plate_mass"  value="0.2304" />   <!-- Density: 4440 kg/m3 -->
+  <property name="wrist_coupling_mass"    value="0.059" />    <!-- Density: 5000 kg/m3 -->
+  <property name="ft_coupling_mass"    value="0.1478" />   <!-- Density: 4070 kg/m3 -->
   <property name="ft_sensor_mass"         value="0.2396" />   <!-- Density: 1750 kg/m3 -->
-  <property name="ft_wrist_plate_mass"    value="0.1478" />   <!-- Density: 4070 kg/m3 -->
+  <property name="robotiq_coupling_mass"  value="0.2304" />   <!-- Density: 4440 kg/m3 -->
   <property name="robotiq_mass"           value="2.438" />
-  <!-- Links COG -->
-  <property name="ft_kraft_plate_cog"     value="-0.192e-3  1.769e-9    6.143e-3" />
-  <property name="ft_robotiq_plate_cog"   value="0.0        0.0         5.644e-3" />
-  <property name="ft_sensor_cog"          value="9.396e-4   0.017       -7.545e-4" />
-  <property name="ft_wrist_plate_cog"     value="-0.057e-3  1.648e-8    17.057e-3" />
-  <!-- Links Inertia -->
-  <macro name="ft_kraft_plate_inertia">
-    <inertia  ixx="8.905e-6"  iyy="8.788e-6"  izz="1.421e-5"
-              ixy="0.0"       ixz="4.509e-8"  iyz="0.0" />
-  </macro>
-  <macro name="ft_robotiq_plate_inertia">
-    <inertia  ixx="9.43e-5"   iyy="9.43e-5"   izz="1.837e-4"
-              ixy="0.0"       ixz="0.0"       iyz="0.0" />
-  </macro>
-  <macro name="ft_sensor_inertia">
-    <inertia  ixx="1.055e-4"  iyy="1.7e-4"    izz="1.076e-4"
-              ixy="-7.262e-7" ixz="6.186e-6"  iyz="6.529e-7" />
-  </macro>
-  <macro name="ft_wrist_plate_inertia">
-    <inertia  ixx="4.686e-5"  iyy="4.663e-5"  izz="8.289e-5"
-              ixy="0.0"       ixz="0.0"       iyz="0.0" />
-  </macro>
-  <macro name="ftsensor" params="name parent">
+  <macro name="ftsensor" params="parent">
     <!-- Links -->
-    <create_link name="${name}ft_kraft_plate" color="black" mesh="${ft_kraft_plate_mesh}" mass="${ft_kraft_plate_mass}" cog="${ft_kraft_plate_cog}" >
-      <ft_kraft_plate_inertia />
+    <create_link name="wrist_coupling" color="white" mesh="${wrist_coupling_mesh}" >
+      <cylinder_collision radius="${wrist_coupling_radius}" length="${wrist_coupling_length}" />
+      <cylinder_inertia radius="${wrist_coupling_radius}" length="${wrist_coupling_length}" mass="${wrist_coupling_mass}"/>
     </create_link>
-    <create_link name="${name}ft_wrist_plate" color="black" mesh="${ft_wrist_plate_mesh}" mass="${ft_wrist_plate_mass}" cog="${ft_wrist_plate_cog}" >
-      <ft_wrist_plate_inertia />
-    </create_link>
-    <create_link name="${name}ft_sensor" color="black" mesh="${ft_sensor_mesh}" mass="${ft_sensor_mass}" cog="${ft_sensor_cog}" >
-      <ft_sensor_inertia />
-    </create_link>
-    <create_link name="${name}ft_robotiq_plate" color="black" mesh="${ft_robotiq_plate_mesh}" mass="${ft_robotiq_plate_mass}" cog="${ft_robotiq_plate_cog}" >
-      <ft_robotiq_plate_inertia />
-    </create_link>
-    <!-- dummy link for attaching end_effector -->
-    <link name="${name}ft_end_effector" />
+    <link name="ft_coupling">
+      <visual>
+        <geometry>
+          <mesh filename="${ft_coupling_mesh}" />
+        </geometry>
+        <material name="white" />
+      </visual>
+      <!-- Align the collision with the mess. It has an offset of 4.7 mm -->
+      <collision>
+        <origin xyz="0 0 ${4.7e-3 + ft_coupling_length/2}" rpy="0 0 0"/>
+        <geometry>
+          <cylinder radius="${ft_coupling_radius}" length="${ft_coupling_length}"/>
+        </geometry>
+      </collision>
+      <inertial>
+        <origin xyz="0 0 ${4.7e-3 + ft_coupling_length/2}" rpy="0 0 0" />
+        <mass value="${ft_coupling_mass}" />
+        <inertia  ixx="${ft_coupling_mass*ft_coupling_radius^2 / 4  + ft_coupling_mass*ft_coupling_length^2 / 12}" ixy="0.0"  ixz="0.0"
+                  iyy="${ft_coupling_mass*ft_coupling_radius^2 / 4  + ft_coupling_mass*ft_coupling_length^2 / 12}" iyz="0.0"
+                  izz="${ft_coupling_mass*ft_coupling_radius^2 / 2}" />
+      </inertial>
+    </link>
+    <link name="ft_sensor">
+      <visual>
+        <origin xyz="0 0 0" rpy="${-pi/2} 0 0"/>
+        <geometry>
+          <mesh filename="${ft_sensor_mesh}" />
+        </geometry>
+        <material name="white" />
+      </visual>
+      <collision>
+        <origin xyz="0 0 ${-ft_sensor_length/2}" rpy="0 0 0"/>
+        <geometry>
+          <cylinder radius="${ft_sensor_radius}" length="${ft_sensor_length}"/>
+        </geometry>
+      </collision>
+      <inertial>
+        <origin xyz="0 0 ${-ft_sensor_length/2}" rpy="0 0 0" />
+        <mass value="${ft_sensor_mass}" />
+        <inertia  ixx="${ft_sensor_mass*ft_sensor_radius^2 / 4  + ft_sensor_mass*ft_sensor_length^2 / 12}" ixy="0.0"  ixz="0.0"
+                  iyy="${ft_sensor_mass*ft_sensor_radius^2 / 4  + ft_sensor_mass*ft_sensor_length^2 / 12}" iyz="0.0"
+                  izz="${ft_sensor_mass*ft_sensor_radius^2 / 2}" />
+      </inertial>
+    </link>
     <!-- Joints -->
-    <joint name="${name}ft_robot_joint" type="fixed">
+    <joint name="ft_robot_joint" type="fixed">
       <origin xyz="0 0 0" rpy="${-pi/2} 0 0" />
       <parent link="${parent}" />
-      <child link="${name}ft_kraft_plate" />
+      <child link="wrist_coupling" />
     </joint>
-    <joint name="${name}ft_wrist_joint" type="fixed">
+    <joint name="ft_wrist_joint" type="fixed">
       <origin xyz="0 0 0" rpy="0 0 0" />
-      <parent link="${name}ft_kraft_plate" />
-      <child link="${name}ft_wrist_plate" />
+      <parent link="wrist_coupling" />
+      <child link="ft_coupling" />
     </joint>
-    <joint name="${name}ft_sensor_joint" type="fixed">
-      <origin xyz="0 0 ${23.7e-3+32.7e-3}" rpy="${-pi/2} 0 0" />
-      <parent link="${name}ft_wrist_plate" />
-      <child link="${name}ft_sensor" />
-    </joint>
-    <joint name="${name}ft_plate_joint" type="fixed">
-      <origin xyz="0 -11e-3 0" rpy="${-pi/2} 0 0" />
-      <parent link="${name}ft_sensor" />
-      <child link="${name}ft_robotiq_plate" />
-    </joint>
-    <joint name="${name}ft_end_joint" type="fixed">
-      <origin xyz="0 0 0" rpy="${-pi/2} 0 0" />
-      <parent link="${name}ft_robotiq_plate" />
-      <child link="${name}ft_end_effector" />
+    <joint name="ft_sensor_joint" type="fixed">
+      <origin xyz="0 0 ${4.7e-3 + ft_coupling_length + ft_sensor_length}" rpy="0 0 0" />
+      <parent link="ft_coupling" />
+      <child link="ft_sensor" />
     </joint>
   </macro>
