Commit message: Improved grips joint limits and fixed four-bar equations

File: grips_description/urdf/serial_arm.xacro (robot description, xacro)
@@ -129,5 +129,5 @@
       <axis xyz="1 0 0" />
       <origin xyz="0 -9.82e-3 ${upper_arm_length}" rpy="0 0 0" />
-      <limit lower="-1.28" upper="${pi/3}" effort="${max_effort}" velocity="${50*pi/180}" />
+      <limit lower="${-40*pi/180}" upper="${70*pi/180}" effort="${max_effort}" velocity="${50*pi/180}" />
       <dynamics damping="10"/>
     </joint>
@@ -137,5 +137,5 @@
       <axis xyz="1 0 0" />
       <origin xyz="0 0.26109 7.5e-3" rpy="0 0 0" />
-      <limit lower="-0.581" upper="1.1" effort="${max_effort}" velocity="${100*pi/180}" />
+      <limit lower="${-35*pi/180}" upper="${65*pi/180}" effort="${max_effort}" velocity="${100*pi/180}" />
       <dynamics damping="${WP_damping}"/>
     </joint>
@@ -145,5 +145,5 @@
       <axis xyz="0 0 1" />
       <origin xyz="0 ${pitch_length} 0" rpy="0 0 0" />
-      <limit lower="-1.01" upper="0.675" effort="${max_effort}" velocity="${115*pi/180}" />
+      <limit lower="${-39*pi/180}" upper="${66*pi/180}" effort="${max_effort}" velocity="${115*pi/180}" />
       <dynamics damping="${WY_damping}"/>
     </joint>

Commit message: Updated WR position limits

File: grips_description/urdf/serial_arm.xacro (robot description, xacro)
@@ -153,5 +153,5 @@
       <axis xyz="0 1 0" />
       <origin xyz="-0.787e-3 ${yaw_length} 0.051331" rpy="0 0 0" />
-      <limit lower="${-pi}" upper="${pi}" effort="${max_effort}" velocity="${200*pi/180}" />
+      <limit lower="${-100*pi/180}" upper="${100*pi/180}" effort="${max_effort}" velocity="${200*pi/180}" />
       <dynamics damping="${WR_damping}"/>
     </joint>
